File: src/cherry.kicad_pcb (KiCad board)
At the start: 2 copper layers, 61.2 x 26.1 mm, 72 parts, among them J1 USB4085-GF-A, J2 PinHeader_1x24, J3 PinHeader_1x06, J4 PinHeader_1x06, J5 PinHeader_1x06, J6 PinHeader_1x24, SW1 RESET, SW2 USER, U1 FT2232HQ, U2 ICE40LP8K-CM81, U3 W25Q32JVSSIQ, U4 TPS62A02, U5 TPS62A02, X1 ASE-12.000MHZ-LC-T

Commit message: 56Q
Parts:
- added D5: USBLC6-2SC6, Cherry:SOT-23-6, F.Cu at (117.5, 86.6)
- U1: value FT2232HQ -> FT2232H-56Q; footprint Cherry:QFN-64-1EP_9x9mm_P0.5mm_EP4.35x4.35mm -> Cherry:QFN-56-1EP_8x8mm_P0.5mm_EP5.9x5.9mm
- U3: footprint Cherry:SOIC-8_3.9x4.9mm_P1.27mm -> Cherry:SOIC-8_5.3x5.3mm_P1.27mm
- X1: value ASE-12.000MHZ-LC-T -> ASE-12.000MHZ-LR-T
- moved C28 1.27 mm to (134.6, 83.8)
- moved R11 1.27 mm to (137.2, 83.8)
- moved R18 1.27 mm to (134.0, 96.5)
- moved R19 1.27 mm to (135.3, 96.5)
- moved R20 1.27 mm to (136.5, 96.5)
- moved R21 1.27 mm to (137.8, 96.5)
Connections:
- net Net-(FB1-Pad2) renamed /VBUS
- U1 pad 1: GND -> unconnected-(U1-EECS-Pad1)
- U1 pad 11: GND -> Net-(U1-~{RESET})
- U1 pad 12: /VCORE -> /FT_SCK
- U1 pad 13: GND -> /FT_MOSI
- U1 pad 14: Net-(U1-~{RESET}) -> /FT_MISO
- U1 pad 15: GND -> unconnected-(U1-ADBUS3-Pad15)
- U1 pad 16: /FT_SCK -> +3V3
- U1 pad 17: /FT_MOSI -> /FT_SS
- U1 pad 18: /FT_MISO -> unconnected-(U1-ADBUS5-Pad18)
- U1 pad 19: unconnected-(U1-ADBUS3-Pad19) -> /CDONE
- U1 pad 2: /CLK_12M -> /VCORE
- U1 pad 20: +3V3 -> /FT_CRESET
- U1 pad 21: /FT_SS -> GND
- U1 pad 23: /CDONE -> unconnected-(U1-ACBUS1-Pad23)
- U1 pad 24: /FT_CRESET -> unconnected-(U1-ACBUS2-Pad24)
- U1 pad 25: GND -> unconnected-(U1-ACBUS3-Pad25)
- U1 pad 3: unconnected-(U1-OSCO-Pad3) -> /CLK_12M
- U1 pad 31: +3V3 -> /VCORE
- U1 pad 32: unconnected-(U1-ACBUS5-Pad32) -> /UART_TX
- U1 pad 33: unconnected-(U1-ACBUS6-Pad33) -> /UART_RX
- U1 pad 35: GND -> unconnected-(U1-BDBUS3-Pad35)
- U1 pad 36: unconnected-(U1-~{SUSPEND}-Pad36) -> +3V3
- U1 pad 37: /VCORE -> unconnected-(U1-BDBUS4-Pad37)
- U1 pad 38: /UART_TX -> unconnected-(U1-BDBUS5-Pad38)
- U1 pad 39: /UART_RX -> unconnected-(U1-BDBUS6-Pad39)
- U1 pad 4: /+3V3A -> unconnected-(U1-OSCO-Pad4)
- U1 pad 41: unconnected-(U1-BDBUS3-Pad41) -> GND
- U1 pad 42: +3V3 -> unconnected-(U1-BCBUS0-Pad42)
- U1 pad 43: unconnected-(U1-BDBUS4-Pad43) -> /VCORE
- U1 pad 44: unconnected-(U1-BDBUS5-Pad44) -> +3V3
- U1 pad 45: unconnected-(U1-BDBUS6-Pad45) -> GND
- U1 pad 47: GND -> unconnected-(U1-BCBUS2-Pad47)
- U1 pad 49: /VCORE -> unconnected-(U1-BCBUS4-Pad49)
- U1 pad 5: GND -> /+3V3A
- U1 pad 51: GND -> unconnected-(U1-BCBUS5-Pad51)
- U1 pad 56: +3V3 -> unconnected-(U1-EECLK-Pad56)
- U1 pad 57: unconnected-(U1-BCBUS5-Pad57) -> GND

Commit message: layout
Parts:
- removed C7: 100nF, Cherry:C_0402_1005Metric
- moved X1 23.5 mm to (135.9, 82.5), turned to 0 degrees
- moved R11 13.3 mm to (133.3, 96.5), turned to 90 degrees
- moved C8 12.8 mm to (128.9, 83.8), turned to 90 degrees
- moved R7 12.1 mm to (128.9, 96.5), turned to -90 degrees
- moved C13 12.0 mm to (124.5, 96.5), turned to -90 degrees
- moved R8 9.61 mm to (130.2, 96.5)
- moved C5 9.55 mm to (121.9, 83.2), turned to 90 degrees
- moved C14 8.13 mm to (125.7, 96.5), turned to -90 degrees
- moved C28 6.98 mm to (127.6, 83.8), turned to 90 degrees
- moved D5 6.14 mm to (112.4, 83.2), turned to 90 degrees
- moved C21 4.61 mm to (146.7, 95.9), turned to -90 degrees
- moved C10 4.58 mm to (123.2, 96.5)
- moved C12 4.45 mm to (123.8, 83.8), turned to 90 degrees
- moved C24 4.19 mm to (147.3, 84.5)
- moved R22 4.07 mm to (128.9, 99.1), turned to 90 degrees
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
Commit message: refactor
Parts:
- R1: value 180k -> 100k
- R2: value 39.2k -> 22k
- U2: renamed from U3; value W25Q32JVSSIQ -> W25Q32JVSSIM
- renumbered C11 to C10, C5 to C11, C13 to C12, C14 to C13, C15 to C14, C16 to C15, C17 to C16, C18 to C17, C19 to C18, C20 to C19, C21 to C20, C22 to C21, C23 to C22, C24 to C23, C25 to C24, C28 to C25, C6 to C5, C8 to C6, C9 to C7, C12 to C8, C10 to C9, J6 to J3, J3 to J4, J4 to J5, J5 to J6, R18 to R14, R19 to R15, R20 to R16, R21 to R17, R22 to R18, R14 to R19, R15 to R20, R16 to R21, R17 to R22, U2 to U3

Commit message: FT2232HL, 4-layer, renumber, pdf
Parts:
- added C17: 100nF, Cherry:C_0402_1005Metric, F.Cu at (120.7, 97.8)
- C26: renamed from C11; value 4.7uF -> 10uF; footprint Cherry:C_0603_1608Metric -> Cherry:C_0805_2012Metric
- C27: footprint Cherry:C_0603_1608Metric -> Cherry:C_0805_2012Metric
- U1: value FT2232H-56Q -> FT2232HL; footprint Cherry:QFN-56-1EP_8x8mm_P0.5mm_EP5.9x5.9mm -> Cherry:LQFP-64_10x10mm_P0.5mm
- moved R12 2.14 mm to (132.4, 98.4)
- moved C26 1.37 mm to (121.9, 81.8)
- moved R7 1.33 mm to (128.9, 97.8)
- moved R8 1.33 mm to (130.2, 97.8)
- moved C12 1.31 mm to (123.2, 97.8)
- moved C14 1.31 mm to (124.5, 97.8)
- moved C15 1.31 mm to (125.7, 97.8)
- moved C16 1.31 mm to (127.0, 97.8)
- moved C8 1.31 mm to (121.9, 97.8)
- moved C10 1.31 mm to (126.4, 82.5)
- moved C11 1.31 mm to (123.8, 82.5)
- moved C13 1.31 mm to (125.1, 82.5)
- moved C25 1.31 mm to (127.6, 82.5)
- moved C9 1.31 mm to (128.9, 82.5)
- moved R18 0.77 mm to (128.9, 99.8)
- renumbered C7 to C10, C8 to C11, C9 to C12, C10 to C13, C12 to C14, C13 to C15, C15 to C16, C16 to C18, C17 to C19, C19 to C20, C20 to C21, C21 to C22, C22 to C23, C23 to C24, C26 to C28, C14 to C5, C18 to C6, C24 to C7, C5 to C8, C6 to C9, R11 to R10, R12 to R11, R10 to R12
Connections:
- U1 pad 1: unconnected-(U1-EECS-Pad1) -> GND
- U1 pad 11: Net-(U1-~{RESET}) -> GND
- U1 pad 12: /FT_SCK -> /VCORE
- U1 pad 13: /FT_MOSI -> GND
- U1 pad 14: /FT_MISO -> Net-(U1-~{RESET})
- U1 pad 15: unconnected-(U1-ADBUS3-Pad15) -> GND
- U1 pad 16: +3V3 -> /FT_SCK
- U1 pad 17: /FT_SS -> /FT_MOSI
- U1 pad 18: unconnected-(U1-ADBUS5-Pad18) -> /FT_MISO
- U1 pad 19: /CDONE -> unconnected-(U1-ADBUS3-Pad19)
- U1 pad 2: /VCORE -> /CLK_12M
- U1 pad 20: /FT_CRESET -> +3V3
- U1 pad 21: GND -> /FT_SS
- U1 pad 23: unconnected-(U1-ACBUS1-Pad23) -> /CDONE
- U1 pad 24: unconnected-(U1-ACBUS2-Pad24) -> /FT_CRESET
- U1 pad 25: unconnected-(U1-ACBUS3-Pad25) -> GND
- U1 pad 3: /CLK_12M -> unconnected-(U1-OSCO-Pad3)
- U1 pad 31: /VCORE -> +3V3
- U1 pad 32: /UART_TX -> unconnected-(U1-ACBUS5-Pad32)
- U1 pad 33: /UART_RX -> unconnected-(U1-ACBUS6-Pad33)
- U1 pad 35: unconnected-(U1-BDBUS3-Pad35) -> GND
- U1 pad 36: +3V3 -> unconnected-(U1-~{SUSPEND}-Pad36)
- U1 pad 37: unconnected-(U1-BDBUS4-Pad37) -> /VCORE
- U1 pad 38: unconnected-(U1-BDBUS5-Pad38) -> /UART_TX
- U1 pad 39: unconnected-(U1-BDBUS6-Pad39) -> /UART_RX
- U1 pad 4: unconnected-(U1-OSCO-Pad4) -> /+3V3A
- U1 pad 41: GND -> unconnected-(U1-BDBUS3-Pad41)
- U1 pad 42: unconnected-(U1-BCBUS0-Pad42) -> +3V3
- U1 pad 43: /VCORE -> unconnected-(U1-BDBUS4-Pad43)
- U1 pad 44: +3V3 -> unconnected-(U1-BDBUS5-Pad44)
- U1 pad 45: GND -> unconnected-(U1-BDBUS6-Pad45)
- U1 pad 47: unconnected-(U1-BCBUS2-Pad47) -> GND
- U1 pad 49: unconnected-(U1-BCBUS4-Pad49) -> /VCORE
- U1 pad 5: /+3V3A -> GND
- U1 pad 51: unconnected-(U1-BCBUS5-Pad51) -> GND
- U1 pad 56: unconnected-(U1-EECLK-Pad56) -> +3V3
- U1 pad 57: GND -> unconnected-(U1-BCBUS5-Pad57)
Other:
- copper layers 2 -> 4
