File: src/cherry.kicad_sch (KiCad schematic)
At the start: 19 parts, among them J1 USB_C, J2 2x20_2.54mm, U1 FT2232HL, U2 ICE40LP8K-CM81, U3 W25Q32JVSSIQ, U4 TPS62A02, U5 TPS62A02, Y1 12MHz

Commit message: wip: current layout state
Parts:
- removed J1: USB_C, symbol Cherry:USB_C_Receptacle_USB2.0
- removed J2: 2x20_2.54mm, symbol Cherry:Conn_02x20_Odd_Even
- removed Y1: 12MHz, symbol Cherry:Crystal
- added C10, C11, C12, C13, C14, C16, C17, C18, C20, C21, C22, C23, C24, C26, C28, C6, C7, C8, C9: 100nF, Cherry:C_0402_1005Metric, symbol Cherry:C
- added C15, C19, C25: 10uF, Cherry:C_0805_2012Metric, symbol Cherry:C
- added C27: 10uF, Cherry:C_0603_1608Metric, symbol Cherry:C
- added C5: 4.7uF, Cherry:C_0603_1608Metric, symbol Cherry:C
- added D1: PWR, Cherry:LED_0603_1608Metric, symbol Cherry:LED
- added D2: CFG, Cherry:LED_0603_1608Metric, symbol Cherry:LED
- added D3: USER0, Cherry:LED_0603_1608Metric, symbol Cherry:LED
- added D4: USER1, Cherry:LED_0603_1608Metric, symbol Cherry:LED
- added FB2: BLM21AG601SH1D, Cherry:L_0805_2012Metric, symbol Cherry:Ferrite_Bead
- added J1: USB4085-GF-A, Cherry:USB_C_Receptacle_GCT_USB4085, symbol Cherry:USB_C_USB4085
- added J2: PinHeader_2x24, Cherry:PinHeader_2x24_P2.54mm_Rows22.86mm, symbol Cherry:PinHeader_2x24
- added R10, R11, R12, R8, R9: 10k, Cherry:R_0402_1005Metric, symbol Cherry:R
- added R13: 100, Cherry:R_0402_1005Metric, symbol Cherry:R
- added R14, R15, R16, R17: 1k, Cherry:R_0402_1005Metric, symbol Cherry:R
- added R5, R6: 5.1k, Cherry:R_0402_1005Metric, symbol Cherry:R
- added R7: 12k, Cherry:R_0402_1005Metric, symbol Cherry:R
- added SW1: RESET, Cherry:SW_Push_1P1T_NO_CK_KMR2, symbol Cherry:SW_Push
- added SW2: USER, Cherry:SW_Push_1P1T_NO_CK_KMR2, symbol Cherry:SW_Push
- added X1: ASE-12.000MHZ-LC-T, Cherry:Oscillator_SMD_Abracon_ASE-4Pin_3.2x2.5mm, symbol Cherry:XO_3225
- C1, C2, C3, C4: footprint (none) -> Cherry:C_0805_2012Metric
- FB1: value FB_600R -> BLM21AG601SH1D; footprint (none) -> Cherry:L_0805_2012Metric
- L1, L2: footprint (none) -> Cherry:L_0805_2012Metric
- R1, R2, R3, R4: footprint (none) -> Cherry:R_0402_1005Metric
- U1: value FT2232HL -> FT2232HQ; footprint (none) -> Cherry:QFN-64-1EP_9x9mm_P0.5mm_EP4.35x4.35mm
- U2: footprint (none) -> Cherry:BGA-81_9x9_8.0x8.0mm_P0.8mm
- U3: footprint (none) -> Cherry:SOIC-8_3.9x4.9mm_P1.27mm
- U4, U5: footprint (none) -> Cherry:SOT-23-6
Connections:
- net +1V2: now also U2.D4 (VCC), U2.E9 (VCC), C17.1, C18.1, C19.1, R13.1; no longer C1.1, C2.1, C3.1, C3.2, C4.2, L1.1, L1.2, L2.1, R1.1, R1.2, R2.1, R2.2, R3.2, R4.1, R4.2, U1.10 (VCCIO_A), U1.13 (~{TRST}), U1.14 (~{RESET}), U1.2 (OSCI), U1.3 (OSCO), U1.4 (VPHY), U1.55 (EECS), U1.56 (EEDATA), U1.57 (EECLK), U1.6 (REF), U1.7 (DM), U1.9 (VPLL), U2.A5 (CDONE), U2.E5 (GND), U2.F7 (SPI_SO), U2.G6 (SPI_SI), U2.G7 (SPI_SCK), U2.G8 (CRESET_B), U2.G9 (GND), U2.H6 (GND), U2.J3 (GND), U3.3 (~{WP}), U3.4 (GND), U4.1 (VIN), U4.3 (SW), U4.4 (FB), U4.5 (EN), U5.1 (VIN), U5.3 (SW), U5.4 (FB), U5.5 (EN)
- net +5V: now also C1.1, C2.1, U4.1 (EN), U4.4 (VIN), U5.1 (EN), U5.4 (VIN), J2.47, J2.48; no longer C1.2, C2.2, FB1.2, U4.2 (GND), U4.6 (MODE), U5.2 (GND), U5.6 (MODE)
- net CDONE: now also U1.23 (ADBUS6), U2.E6 (CDONE), D2.1 (K), R10.2; no longer U1.41 (BDBUS3), U1.43 (BDBUS4), U1.59 (BCBUS4), U1.60 (BCBUS5), U1.61 (BCBUS6), U1.62 (BCBUS7), U1.63 (~{PWREN}), U2.A4 (GND), U2.B1 (VCCIO_0), U2.B9 (GND), U2.C4 (IOB_34), U2.C5 (IOB_35), U2.C6 (GND), U2.H9 (VCCIO_2), U3.5 (DI), U3.6 (CLK)
- net GPIO_0: now also U2.B1 (IOL_3A), J2.1; no longer U2.C7 (IOB_41), U2.C8 (IOB_42), U2.C9 (IOB_43), U2.D1 (IOB_44), U2.D2 (IOB_45), U2.D4 (IOB_46), U2.D5 (IOB_48), U2.D6 (IOB_49), U2.D7 (IOB_51), U2.D8 (IOB_54)
- net UART_RX: now also U1.39 (BDBUS1), U2.H9 (IOR_111)
- net USB_DM: now also U1.7 (DM), J1.A7 (D-), J1.B7 (D-); no longer U1.26 (GND), U1.36 (GND), U1.64 (GND)
- net GND: now reaches U1.1 (GND)
- net GND: now also C1.2, C2.2, C3.2, C4.2, R2.2, R4.2, U1.10 (AGND), U1.11 (GND), U1.13 (TEST), U1.15 (GND), U1.25 (GND), U1.35 (GND), U1.47 (GND), U1.5 (GND), U1.51 (GND), U1.65 (GND), U2.F4 (GND), U2.F5 (GND), U2.F6 (GND), U2.F9 (GND), U3.4 (GND), U4.2 (GND), U5.2 (GND), C10.2, C11.2, C12.2, C13.2, C14.2, C15.2, C16.2, C17.2, C18.2, C19.2, C20.2, C21.2, C22.2, C23.2, C24.2, C25.2, C28.2, C5.2, C6.2, C7.2, C8.2, C9.2, D3.1 (K), D4.1 (K), J1.A1 (GND), J1.A12 (GND), J1.B1 (GND), J1.B12 (GND), J1.SH (SHIELD), J2.13, J2.18, J2.3, J2.31, J2.36, J2.41, J2.46, J2.8, R14.2, R5.2, R6.2, R7.2, SW1.2, SW2.2, X1.2 (GND)
- net VCORE: now reaches U1.12 (VCORE)
- net VCORE: now also U1.37 (VCORE), U1.49 (VREGOUT), U1.64 (VCORE), C10.1, C11.1, C5.1
- net SPI_SCK: now reaches U1.16 (ADBUS0)
- net SPI_SCK: now also U2.G7 (IOB_107_SCK), U3.6 (CLK)
- net SPI_MOSI: now reaches U1.17 (ADBUS1)
- net SPI_MOSI: now also U2.G6 (IOB_105_SDO), U3.5 (DI)
- net SPI_MISO: now reaches U1.18 (ADBUS2)
- net SPI_MISO: now also U2.H7 (IOB_106_SDI), U3.2 (DO)
- net SPI_SS: now reaches U1.21 (ADBUS4)
- net SPI_SS: now also U2.F7 (IOB_108_SS), U3.1 (~{CS}), R11.2
- net CRESET_B: now reaches U1.24 (ADBUS7)
- net CRESET_B: now also U2.H6 (CRESET_B), J2.38, R9.2, SW1.1
- net UART_TX: now reaches U1.38 (BDBUS0)
- net UART_TX: now also U2.J4 (IOB_70)
- net +3V3: now reaches U1.50 (VREGIN)
- net +3V3: now also C3.1, L1.2, R1.1, U1.20 (VCCIO), U1.31 (VCCIO), U1.42 (VCCIO), U1.56 (VCCIO), U2.A5 (VCCIO_0), U2.C6 (VCCIO_1), U2.C8 (VPP_2V5), U2.H3 (VCCIO_3), U2.H8 (VCC_SPI), U2.J5 (VCCIO_2), U3.3 (~{WP}), U3.7 (~{HOLD}), U3.8 (VCC), C12.1, C16.1, C20.1, C21.1, C22.1, C23.1, C24.1, C25.1, C28.1, C6.1, C7.1, C8.1, C9.1, D1.2 (A), FB2.1, J2.44, R10.1, R11.1, R12.1, R15.1, R8.1, R9.1, X1.1 (EN), X1.4 (VDD)
- net USB_DP: now reaches U1.8 (DP)
- net USB_DP: now also J1.A6 (D+), J1.B6 (D+)
- net GPIO_27: now reaches U2.A2 (IOT_221)
- net GPIO_27: now also J2.45
- net GPIO_25: now reaches U2.A3 (IOT_217)
- net GPIO_25: now also J2.42
- net GPIO_20: now reaches U2.A6 (IOT_185)
- net GPIO_20: now also J2.34
- net GPIO_18: now reaches U2.A7 (IOT_177)
- net GPIO_18: now also J2.32
- net GPIO_16: now reaches U2.A8 (IOT_174)
- net GPIO_16: now also J2.29
- net GPIO_32: now reaches U2.A9 (IOR_116)
- net GPIO_32: now also J2.25
- net GPIO_26: now reaches U2.B3 (IOT_218)
- net GPIO_26: now also J2.43
- net GPIO_24: now reaches U2.B4 (IOT_211)
- net GPIO_24: now also J2.40
- net GPIO_22: now reaches U2.B5 (IOT_188)
- net GPIO_22: now also J2.37
- net GPIO_21: now reaches U2.B6 (IOT_183)
- net GPIO_21: now also J2.35
- net GPIO_19: now reaches U2.B7 (IOT_180)
- net GPIO_19: now also J2.33
- net GPIO_17: now reaches U2.B8 (IOT_170)
- net GPIO_17: now also J2.30
- net GPIO_1: now reaches U2.C1 (IOL_3B)
- net GPIO_1: now also J2.2
- net GPIO_3: now reaches U2.C2 (IOL_2A)
- net GPIO_3: now also J2.5
- net GPIO_8: now reaches U2.D9 (IOR_119)
- net GPIO_8: now also J2.11
- net GPIO_6: now reaches U2.E1 (IOL_10B)
- net GPIO_6: now also J2.9
- net GPIO_7: now reaches U2.E2 (IOL_13A)
- net GPIO_7: now also J2.10
- net GPIO_28: now reaches U2.E7 (IOR_118)
- net GPIO_28: now also J2.21
- net GPIO_29: now reaches U2.F8 (IOR_113)
- net GPIO_29: now also J2.22
- net GPIO_13: now reaches U2.J1 (IOB_55)
- net GPIO_13: now also J2.17
- new net: R7.1, U1.6 (REF)
- new net: D3.2 (A), R16.2
- new net: J1.A5 (CC1), R5.1
- new net: L1.1, U4.3 (SW)
- new net: R1.2, R2.1, U4.6 (FB)
- new net: FB1.2, J1.A4 (VBUS), J1.A9 (VBUS), J1.B4 (VBUS), J1.B9 (VBUS)
- new net: D2.2 (A), R15.2
- new net: J1.B5 (CC2), R6.1
- new net: R3.2, R4.1, U5.6 (FB)
- new net: L2.1, U5.3 (SW)
- new net: D1.1 (K), R14.1
- new net: D4.2 (A), R17.2
- new net +3V3A: C13.1, C14.1, C15.1, FB2.2, U1.4 (VPHY), U1.9 (VPLL)
- new net BTN: R12.2, SW2.1, U2.H4 (IOB_82_GBIN4)
- new net CLK_12M: U1.2 (OSCI), U2.C4 (IOT_198_GBIN0), X1.3 (OUT)
- new net FT_RESET: R8.2, U1.14 (~{RESET})
- new net GNDPLL: C26.2, C27.2, U2.J6 (GNDPLL0)
- new net GPIO_10: J2.14, U2.F1 (IOL_22A)
- new net GPIO_11: J2.15, U2.G9 (IOR_112)
- new net GPIO_12: J2.16, U2.H1 (IOB_54)
- new net GPIO_14: J2.19, U2.J2 (IOB_56)
- new net GPIO_15: J2.20, U2.J3 (IOB_57)
- new net GPIO_2: J2.4, U2.B2 (IOL_2B)
- new net GPIO_23: J2.39, U2.A4 (IOT_208)
- new net GPIO_30: J2.23, U2.G8 (IOR_114)
- new net GPIO_31: J2.24, U2.E8 (IOR_140_GBIN3)
- new net GPIO_33: J2.26, U2.B9 (IOR_120)
- new net GPIO_34: J2.27, U2.D6 (IOR_115)
- new net GPIO_35: J2.28, U2.D7 (IOR_117)
- new net GPIO_4: J2.6, U2.D1 (IOL_10A)
- new net GPIO_5: J2.7, U2.D2 (IOL_7A)
- new net GPIO_9: J2.12, U2.C9 (IOR_148)
- new net LED0: R16.1, U2.J8 (IOR_109)
- new net LED1: R17.1, U2.J9 (IOR_110)
- new net VCCPLL: C26.1, C27.1, R13.2, U2.J7 (VCCPLL0)
- no-connect marks 0 -> 52
Other:
- note added: "12MHz Clock"
- note added: "Buck 5V->1.2V"
- note added: "Buck 5V->3.3V"
- note added: "Config / User"
- note added: "Decoupling - FT2232H"
- note added: "Decoupling - iCE40"
- note added: "FPGA - iCE40LP8K-CM81"
- note added: "GPIO Header (RPi Pico compatible)"
- note added: "LEDs"
- note added: "PLL Filter"
- note added: "SPI Flash"
- note added: "USB Bridge - FT2232HL"
- note added: "USB-C"
