File: src/cherry.kicad_sch (KiCad schematic)
At the start: 63 parts, among them J1 USB4085-GF-A, J2 PinHeader_2x24, SW1 RESET, SW2 USER, U1 FT2232HQ, U2 ICE40LP8K-CM81, U3 W25Q32JVSSIQ, U4 TPS62A02, U5 TPS62A02, X1 ASE-12.000MHZ-LC-T

Commit message: wip
Parts:
- added unit 2 of J2
- added J3, J4, J5: PinHeader_1x06, Connector_PinHeader_2.54mm:PinHeader_1x06_P2.54mm_Vertical, symbol Cherry:PinHeader_1x06
Connections:
- net +3V3: now also J2.44; no longer J2.44
- net +5V: now also J2.47, J2.48; no longer J2.47, J2.48
- net CDONE: now also D2.1 (K)
- net CRESET_B: now also J2.38; no longer J2.38
- net GND: now also J2.31, J2.36, J2.41, J2.46; no longer J2.31, J2.36, J2.41, J2.46
- net GPIO_16: now also J2.29; no longer J2.29
- net GPIO_17: now also J2.30; no longer J2.30
- net GPIO_18: now also J2.32; no longer J2.32
- net GPIO_19: now also J2.33; no longer J2.33
- net GPIO_20: now also J2.34; no longer J2.34
- net GPIO_21: now also J2.35; no longer J2.35
- net GPIO_22: now also J2.37; no longer J2.37
- net GPIO_23: now also J2.39; no longer J2.39
- net GPIO_24: now also J2.40; no longer J2.40
- net GPIO_25: now also J2.42; no longer J2.42
- net GPIO_26: now also J2.43; no longer J2.43
- net GPIO_27: now also J2.45; no longer J2.45
- net GPIO_32: now also J2.25; no longer J2.25
- net GPIO_33: now also J2.26; no longer J2.26
- net GPIO_34: now also J2.27; no longer J2.27
- net GPIO_35: now also J2.28; no longer J2.28
- no-connect marks 52 -> 70
