File: src/cherry.kicad_sch (KiCad schematic)
At the start: 67 parts, among them J1 USB4085-GF-A, J2 PinHeader_1x24, J3 PinHeader_1x06, J4 PinHeader_1x06, J5 PinHeader_1x06, J6 PinHeader_1x24, SW1 RESET, SW2 USER, U1 FT2232HQ, U2 ICE40LP8K-CM81, U3 W25Q32JVSSIQ, U4 TPS62A02, U5 TPS62A02, X1 ASE-12.000MHZ-LC-T

Commit message: wip
Parts:
- added R18, R19, R20, R21: 470, Cherry:R_0402_1005Metric, symbol Cherry:R
- added R22: 1k, Cherry:R_0402_1005Metric, symbol Cherry:R
- J2, J6: footprint Connector_PinHeader_2.54mm:PinHeader_1x24_P2.54mm_Vertical -> Cherry:PinHeader_1x24_P2.54mm
- J3, J4, J5: footprint Connector_PinHeader_2.54mm:PinHeader_1x06_P2.54mm_Vertical -> Cherry:PinHeader_1x06_P2.54mm
- R10: value 10k -> 1k
Connections:
- net +3V3: now also J2.2, J6.23; no longer J6.9, R15.1
- net +5V: now also J2.1, J6.24; no longer J6.5, J6.6
- net CDONE: now also R15.1; no longer D2.1 (K)
- net CRESET_B: now also J2.6, R22.2; no longer J6.15, U1.24 (ADBUS7)
- net GND: now also D2.1 (K), J2.3, J2.4, J2.5, J5.6 (Pin_6), J6.19, J6.20, J6.21; no longer J2.12, J2.17, J2.22, J2.7, J6.12, J6.17, J6.7
- net GPIO_1: now also J2.7, U2.G8 (IOR_114); no longer J2.6, U2.C1 (IOL_3B)
- net GPIO_10: now also J2.16, U2.E1 (IOL_10B); no longer J2.18, U2.F1 (IOL_22A)
- net GPIO_11: now also J2.17, U2.E2 (IOL_13A); no longer J2.19, U2.G9 (IOR_112)
- net GPIO_12: now also J2.18, U2.D9 (IOR_119); no longer J2.20, U2.H1 (IOB_54)
- net GPIO_13: now also J2.19, U2.C9 (IOR_148); no longer J2.21, U2.J1 (IOB_55)
- net GPIO_14: now also J2.20, U2.F1 (IOL_22A); no longer J2.23, U2.J2 (IOB_56)
- net GPIO_15: now also J2.21, U2.G9 (IOR_112); no longer J2.24, U2.J3 (IOB_57)
- net GPIO_16: now also J2.22, U2.H1 (IOB_54); no longer J6.24, U2.A8 (IOT_174)
- net GPIO_17: now also J2.23, U2.J1 (IOB_55); no longer J6.23, U2.B8 (IOT_170)
- net GPIO_18: now also J2.24, U2.J2 (IOB_56); no longer J6.21, U2.A7 (IOT_177)
- net GPIO_19: now also J6.1, U2.A9 (IOR_116); no longer J6.20, U2.B7 (IOT_180)
- net GPIO_2: now also U2.F8 (IOR_113); no longer U2.B2 (IOL_2B)
- net GPIO_20: now also J6.2, U2.B9 (IOR_120); no longer J6.19, U2.A6 (IOT_185)
- net GPIO_21: now also J6.3, U2.D6 (IOR_115); no longer J6.18, U2.B6 (IOT_183)
- net GPIO_22: now also J6.4, U2.D7 (IOR_117); no longer J6.16, U2.B5 (IOT_188)
- net GPIO_23: now also J6.5, U2.A2 (IOT_221); no longer J6.14, U2.A4 (IOT_208)
- net GPIO_24: now also J6.6, U2.B3 (IOT_218); no longer J6.13, U2.B4 (IOT_211)
- net GPIO_25: now also J6.7; no longer J6.11
- net GPIO_26: now also J6.8, U2.B4 (IOT_211); no longer J6.10, U2.B3 (IOT_218)
- net GPIO_27: now also J6.9, U2.A4 (IOT_208); no longer J6.8, U2.A2 (IOT_221)
- net GPIO_28: now also J6.10, U2.E8 (IOR_140_GBIN3); no longer J2.4, U2.E7 (IOR_118)
- net GPIO_29: now also J6.11, U2.B5 (IOT_188); no longer J2.3, U2.F8 (IOR_113)
- net GPIO_3: now also U2.E7 (IOR_118); no longer U2.C2 (IOL_2A)
- net GPIO_30: now also J6.12, U2.B6 (IOT_183); no longer J2.2, U2.G8 (IOR_114)
- net GPIO_31: now also J6.13, U2.A6 (IOT_185); no longer J2.1, U2.E8 (IOR_140_GBIN3)
- net GPIO_32: now also J6.14, U2.B7 (IOT_180); no longer J6.1, U2.A9 (IOR_116)
- net GPIO_33: now also J6.15, U2.A7 (IOT_177); no longer J6.2, U2.B9 (IOR_120)
- net GPIO_34: now also J6.16, U2.B8 (IOT_170); no longer J6.3, U2.D6 (IOR_115)
- net GPIO_35: now also J6.17, U2.A8 (IOT_174); no longer J6.4, U2.D7 (IOR_117)
- net GPIO_4: now also U2.B1 (IOL_3A); no longer U2.D1 (IOL_10A)
- net GPIO_5: now also U2.C1 (IOL_3B); no longer U2.D2 (IOL_7A)
- net GPIO_6: now also J2.12, U2.B2 (IOL_2B); no longer J2.13, U2.E1 (IOL_10B)
- net GPIO_7: now also J2.13, U2.C2 (IOL_2A); no longer J2.14, U2.E2 (IOL_13A)
- net GPIO_8: now also J2.14, U2.D1 (IOL_10A); no longer J2.15, U2.D9 (IOR_119)
- net GPIO_9: now also J2.15, U2.D2 (IOL_7A); no longer J2.16, U2.C9 (IOR_148)
- net SPI_MISO: now also R20.2; no longer U1.18 (ADBUS2)
- net SPI_MOSI: now also R19.2; no longer U1.17 (ADBUS1)
- net SPI_SCK: now also R18.2; no longer U1.16 (ADBUS0)
- net SPI_SS: now also R21.2; no longer U1.21 (ADBUS4)
- net GPIO_49: now reaches J5.1 (Pin_1)
- net GPIO_49: now also U2.G3 (IOL_24A)
- net GPIO_50: now reaches J5.2 (Pin_2)
- net GPIO_50: now also U2.G4 (IOB_81_GBIN5)
- net GPIO_51: now reaches J5.3 (Pin_3)
- net GPIO_51: now also U2.H2 (IOL_26B)
- net GPIO_52: now reaches J5.4 (Pin_4)
- net GPIO_52: now also U2.G5 (IOB_103_CBSEL0)
- net GPIO_53: now reaches J5.5 (Pin_5)
- net GPIO_53: now also U2.H5 (IOB_104_CBSEL1)
- net GPIO_43: now reaches J4.1 (Pin_1)
- net GPIO_43: now also U2.A1 (IOT_224)
- net GPIO_44: now reaches J4.2 (Pin_2)
- net GPIO_44: now also U2.C5 (IOT_197_GBIN1)
- net GPIO_45: now reaches J4.3 (Pin_3)
- net GPIO_45: now also U2.D5 (IOT_212)
- net GPIO_46: now reaches J4.4 (Pin_4)
- net GPIO_46: now also U2.E5 (IOT_214)
- net GPIO_47: now reaches J4.5 (Pin_5)
- net GPIO_47: now also U2.D8 (IOR_141_GBIN2)
- net GPIO_48: now reaches J4.6 (Pin_6)
- net GPIO_48: now also U2.C3 (IOL_7B)
- net GPIO_37: now reaches U2.D3 (IOL_13B_GBIN7)
- net GPIO_37: now also J3.1 (Pin_1)
- net GPIO_38: now reaches U2.E3 (IOL_14A_GBIN6)
- net GPIO_38: now also J3.2 (Pin_2)
- net GPIO_39: now reaches U2.E4 (IOL_14B)
- net GPIO_39: now also J3.3 (Pin_3)
- net GPIO_40: now reaches U2.F3 (IOL_22B)
- net GPIO_40: now also J3.4 (Pin_4)
- net GPIO_41: now reaches U2.G1 (IOL_24B)
- net GPIO_41: now also J3.5 (Pin_5)
- net GPIO_42: now reaches U2.G2 (IOL_26A)
- net GPIO_42: now also J3.6 (Pin_6)
- removed net GPIO_0: J2.5, U2.B1 (IOL_3A)
- new net FT_CRESET: R22.1, U1.24 (ADBUS7)
- new net FT_MISO: R20.1, U1.18 (ADBUS2)
- new net FT_MOSI: R19.1, U1.17 (ADBUS1)
- new net FT_SCK: R18.1, U1.16 (ADBUS0)
- new net FT_SS: R21.1, U1.21 (ADBUS4)
- new net GPIO_36: J6.18, U2.J3 (IOB_57)
- no-connect marks 70 -> 35
Other:
- note added: "LED"
- note added: "Switch"
- note removed: "Config / User"
- note removed: "LEDs"
- moved on the sheet: D1, D2, D3, D4, J2, J3, J4, J5, J6, R12, R14, R15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

Commit message: passive
Connections:
- net BTN: now also U2.C4 (IOT_198_GBIN0); no longer U2.H4 (IOB_82_GBIN4)
- net CLK_12M: now also U2.G4 (IOB_81_GBIN5); no longer U2.C4 (IOT_198_GBIN0)
- net GPIO_1: now also U2.C2 (IOL_2A); no longer U2.G8 (IOR_114)
- net GPIO_10: now also U2.D3 (IOL_13B_GBIN7); no longer U2.E1 (IOL_10B)
- net GPIO_11: now also U2.E3 (IOL_14A_GBIN6); no longer U2.E2 (IOL_13A)
- net GPIO_12: now also U2.E4 (IOL_14B); no longer U2.D9 (IOR_119)
- net GPIO_13: now also U2.F1 (IOL_22A); no longer U2.C9 (IOR_148)
- net GPIO_14: now also U2.F3 (IOL_22B); no longer U2.F1 (IOL_22A)
- net GPIO_15: now also U2.G3 (IOL_24A); no longer U2.G9 (IOR_112)
- net GPIO_16: now also U2.G1 (IOL_24B); no longer U2.H1 (IOB_54)
- net GPIO_17: now also U2.G2 (IOL_26A); no longer U2.J1 (IOB_55)
- net GPIO_18: now also U2.H2 (IOL_26B); no longer U2.J2 (IOB_56)
- net GPIO_19: now also U2.B8 (IOT_170); no longer U2.A9 (IOR_116)
- net GPIO_2: now also U2.B2 (IOL_2B); no longer U2.F8 (IOR_113)
- net GPIO_20: now also U2.A8 (IOT_174); no longer U2.B9 (IOR_120)
- net GPIO_21: now also U2.A7 (IOT_177); no longer U2.D6 (IOR_115)
- net GPIO_22: now also U2.B7 (IOT_180); no longer U2.D7 (IOR_117)
- net GPIO_23: now also U2.B6 (IOT_183); no longer U2.A2 (IOT_221)
- net GPIO_24: now also U2.A6 (IOT_185); no longer U2.B3 (IOT_218)
- net GPIO_25: now also U2.B5 (IOT_188); no longer U2.A3 (IOT_217)
- net GPIO_26: now also U2.C5 (IOT_197_GBIN1); no longer U2.B4 (IOT_211)
- net GPIO_28: now also U2.B4 (IOT_211); no longer U2.E8 (IOR_140_GBIN3)
- net GPIO_29: now also U2.D5 (IOT_212); no longer U2.B5 (IOT_188)
- net GPIO_3: now also U2.B1 (IOL_3A); no longer U2.E7 (IOR_118)
- net GPIO_30: now also U2.E5 (IOT_214); no longer U2.B6 (IOT_183)
- net GPIO_31: now also U2.A3 (IOT_217); no longer U2.A6 (IOT_185)
- net GPIO_32: now also U2.B3 (IOT_218); no longer U2.B7 (IOT_180)
- net GPIO_33: now also U2.A2 (IOT_221); no longer U2.A7 (IOT_177)
- net GPIO_34: now also U2.A1 (IOT_224); no longer U2.B8 (IOT_170)
- net GPIO_35: now also U2.H1 (IOB_54); no longer U2.A8 (IOT_174)
- net GPIO_36: now also U2.J1 (IOB_55); no longer U2.J3 (IOB_57)
- net GPIO_37: now also U2.J2 (IOB_56); no longer U2.D3 (IOL_13B_GBIN7)
- net GPIO_38: now also U2.J3 (IOB_57); no longer U2.E3 (IOL_14A_GBIN6)
- net GPIO_39: now also U2.H4 (IOB_82_GBIN4); no longer U2.E4 (IOL_14B)
- net GPIO_4: now also U2.C1 (IOL_3B); no longer U2.B1 (IOL_3A)
- net GPIO_40: now also U2.G5 (IOB_103_CBSEL0); no longer U2.F3 (IOL_22B)
- net GPIO_41: now also U2.H5 (IOB_104_CBSEL1); no longer U2.G1 (IOL_24B)
- net GPIO_42: now also U2.G9 (IOR_112); no longer U2.G2 (IOL_26A)
- net GPIO_43: now also U2.F8 (IOR_113); no longer U2.A1 (IOT_224)
- net GPIO_44: now also U2.G8 (IOR_114); no longer U2.C5 (IOT_197_GBIN1)
- net GPIO_45: now also U2.D6 (IOR_115); no longer U2.D5 (IOT_212)
- net GPIO_46: now also U2.A9 (IOR_116); no longer U2.E5 (IOT_214)
- net GPIO_47: now also U2.D7 (IOR_117); no longer U2.D8 (IOR_141_GBIN2)
- net GPIO_48: now also U2.E7 (IOR_118); no longer U2.C3 (IOL_7B)
- net GPIO_49: now also U2.D9 (IOR_119); no longer U2.G3 (IOL_24A)
- net GPIO_5: now also U2.D2 (IOL_7A); no longer U2.C1 (IOL_3B)
- net GPIO_50: now also U2.B9 (IOR_120); no longer U2.G4 (IOB_81_GBIN5)
- net GPIO_51: now also U2.E8 (IOR_140_GBIN3); no longer U2.H2 (IOL_26B)
- net GPIO_52: now also U2.D8 (IOR_141_GBIN2); no longer U2.G5 (IOB_103_CBSEL0)
- net GPIO_53: now also U2.C9 (IOR_148); no longer U2.H5 (IOB_104_CBSEL1)
- net GPIO_6: now also U2.C3 (IOL_7B); no longer U2.B2 (IOL_2B)
- net GPIO_7: now also U2.D1 (IOL_10A); no longer U2.C2 (IOL_2A)
- net GPIO_8: now also U2.E1 (IOL_10B); no longer U2.D1 (IOL_10A)
- net GPIO_9: now also U2.E2 (IOL_13A); no longer U2.D2 (IOL_7A)
- net LED0: now also U2.J4 (IOB_70); no longer U2.J8 (IOR_109)
- net UART_TX: now also U2.J8 (IOR_109); no longer U2.J4 (IOB_70)

Commit message: layout
Other:
- moved on the sheet: R5, R6
Changed lines of the file:
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@@
 	(wire
 		(pts
-			(xy 54.61 210.82) (xy 83.82 210.82)
+			(xy 54.61 210.82) (xy 64.77 210.82)
 		)
 		(stroke
@@
 	(wire
 		(pts
-			(xy 83.82 223.52) (xy 83.82 224.79)
+			(xy 64.77 223.52) (xy 64.77 224.79)
 		)
 		(stroke
@@
 	(wire
 		(pts
-			(xy 68.58 213.36) (xy 68.58 215.9)
+			(xy 71.12 213.36) (xy 71.12 215.9)
 		)
 		(stroke
@@
 	(wire
 		(pts
-			(xy 54.61 213.36) (xy 68.58 213.36)
+			(xy 54.61 213.36) (xy 71.12 213.36)
 		)
 		(stroke
@@
 	(wire
 		(pts
-			(xy 83.82 210.82) (xy 83.82 215.9)
+			(xy 64.77 210.82) (xy 64.77 215.9)
 		)
 		(stroke
@@
 	(wire
 		(pts
-			(xy 68.58 223.52) (xy 68.58 224.79)
+			(xy 71.12 223.52) (xy 71.12 224.79)
 		)
 		(stroke
@@
 	(symbol
 		(lib_id "Cherry:R")
-		(at 83.82 219.71 0)
+		(at 64.77 219.71 0)
 		(unit 1)
 		(body_style 1)
@@
 		(dnp no)
 		(property "Reference" "R5"
-			(at 80.37 218.01 0)
+			(at 61.32 218.01 0)
 			(show_name no)
 			(do_not_autoplace no)
@@
 		)
 		(property "Value" "5.1k"
-			(at 79.32 221.41 0)
+			(at 60.27 221.41 0)
 			(show_name no)
 			(do_not_autoplace no)
@@
 		)
 		(property "Footprint" "Cherry:R_0402_1005Metric"
-			(at 83.82 219.71 0)
+			(at 64.77 219.71 0)
 			(hide yes)
 			(show_name no)
@@
 		)
 		(property "Datasheet" ""
-			(at 83.82 219.71 0)
+			(at 64.77 219.71 0)
 			(show_name no)
 			(do_not_autoplace no)
@@
 		)
 		(property "Description" ""
-			(at 83.82 219.71 0)
+			(at 64.77 219.71 0)
 			(show_name no)
 			(do_not_autoplace no)
@@
 	(symbol
 		(lib_id "Cherry:GND")
-		(at 68.58 224.79 0)
+		(at 71.12 224.79 0)
 		(unit 1)
 		(body_style 1)
@@
 		(dnp no)
 		(property "Reference" "#PWR0021"
-			(at 68.58 222.25 0)
+			(at 71.12 222.25 0)
 			(hide yes)
 			(show_name no)
@@
 		)
 		(property "Value" "GND"
-			(at 68.58 228.88 0)
+			(at 71.12 228.88 0)
 			(show_name no)
 			(do_not_autoplace no)
@@
 		)
 		(property "Footprint" ""
-			(at 68.58 224.79 0)
+			(at 71.12 224.79 0)
 			(show_name no)
 			(do_not_autoplace no)
@@
 		)
 		(property "Datasheet" ""
-			(at 68.58 224.79 0)
+			(at 71.12 224.79 0)
 			(show_name no)
 			(do_not_autoplace no)
@@
 		)
 		(property "Description" ""
-			(at 68.58 224.79 0)
+			(at 71.12 224.79 0)
 			(show_name no)
 			(do_not_autoplace no)
@@
 	(symbol
 		(lib_id "Cherry:R")
-		(at 68.58 219.71 0)
+		(at 71.12 219.71 0)
 		(unit 1)
 		(body_style 1)
@@
 		(dnp no)
 		(property "Reference" "R6"
-			(at 72.03 218.01 0)
+			(at 74.57 218.01 0)
 			(show_name no)
 			(do_not_autoplace no)
@@
 		)
 		(property "Value" "5.1k"
-			(at 73.08 221.41 0)
+			(at 75.62 221.41 0)
 			(show_name no)
 			(do_not_autoplace no)
@@
 		)
 		(property "Footprint" "Cherry:R_0402_1005Metric"
-			(at 68.58 219.71 0)
+			(at 71.12 219.71 0)
 			(hide yes)
 			(show_name no)
@@
 		)
 		(property "Datasheet" ""
-			(at 68.58 219.71 0)
+			(at 71.12 219.71 0)
 			(show_name no)
 			(do_not_autoplace no)
@@
 		)
 		(property "Description" ""
-			(at 68.58 219.71 0)
+			(at 71.12 219.71 0)
 			(show_name no)
 			(do_not_autoplace no)
@@
 	(symbol
 		(lib_id "Cherry:GND")
-		(at 83.82 224.79 0)
+		(at 64.77 224.79 0)
 		(unit 1)
 		(body_style 1)
@@
 		(dnp no)
 		(property "Reference" "#PWR0019"
-			(at 83.82 222.25 0)
+			(at 64.77 222.25 0)
 			(hide yes)
 			(show_name no)
@@
 		)
 		(property "Value" "GND"
-			(at 83.82 228.88 0)
+			(at 64.77 228.88 0)
 			(show_name no)
 			(do_not_autoplace no)
@@
 		)
 		(property "Footprint" ""
-			(at 83.82 224.79 0)
+			(at 64.77 224.79 0)
 			(show_name no)
 			(do_not_autoplace no)
@@
 		)
 		(property "Datasheet" ""
-			(at 83.82 224.79 0)
+			(at 64.77 224.79 0)
 			(show_name no)
 			(do_not_autoplace no)
@@
 		)
 		(property "Description" ""
-			(at 83.82 224.79 0)
+			(at 64.77 224.79 0)
 			(show_name no)
 			(do_not_autoplace no)

Commit message: 56Q
Parts:
- added D5: USBLC6-2SC6, Cherry:SOT-23-6, symbol Cherry:USBLC6-2SC6
- U1: value FT2232HQ -> FT2232H-56Q; footprint Cherry:QFN-64-1EP_9x9mm_P0.5mm_EP4.35x4.35mm -> Cherry:QFN-56-1EP_8x8mm_P0.5mm_EP5.9x5.9mm; symbol Cherry:FT2232HL -> Cherry:FT2232H-56Q
- U3: footprint Cherry:SOIC-8_3.9x4.9mm_P1.27mm -> Cherry:SOIC-8_5.3x5.3mm_P1.27mm
- X1: value ASE-12.000MHZ-LC-T -> ASE-12.000MHZ-LR-T
Connections:
- net +3V3: now also U1.16 (VCCIO), U1.36 (VCCIO), U1.44 (VREGIN); no longer U1.20 (VCCIO), U1.31 (VCCIO), U1.42 (VCCIO), U1.56 (VCCIO)
- net +3V3A: now also U1.5 (VPHY); no longer U1.4 (VPHY)
- net CDONE: now also U1.19 (ADBUS6); no longer U1.23 (ADBUS6)
- net CLK_12M: now also U1.3 (OSCI); no longer U1.2 (OSCI)
- net FT_CRESET: now also U1.20 (ADBUS7); no longer U1.24 (ADBUS7)
- net FT_MISO: now also U1.14 (ADBUS2); no longer U1.18 (ADBUS2)
- net FT_MOSI: now also U1.13 (ADBUS1); no longer U1.17 (ADBUS1)
- net FT_SCK: now also U1.12 (ADBUS0); no longer U1.16 (ADBUS0)
- net FT_SS: now also U1.17 (ADBUS4); no longer U1.21 (ADBUS4)
- net GND: now also U1.21 (GND), U1.41 (GND), U1.45 (GND), U1.57 (GND), D5.2 (GND); no longer U1.1 (GND), U1.11 (GND), U1.13 (TEST), U1.15 (GND), U1.25 (GND), U1.35 (GND), U1.47 (GND), U1.5 (GND), U1.51 (GND), U1.65 (GND)
- net UART_RX: now also U1.33 (BDBUS1); no longer U1.39 (BDBUS1)
- net UART_TX: now also U1.32 (BDBUS0); no longer U1.38 (BDBUS0)
- net USB_DM: now also D5.1 (I/O1), D5.6 (I/O1)
- net USB_DP: now also D5.3 (I/O2), D5.4 (I/O2)
- net VCORE: now also U1.2 (VCORE), U1.31 (VCORE), U1.43 (VREGOUT); no longer U1.12 (VCORE), U1.37 (VCORE), U1.49 (VREGOUT), U1.64 (VCORE)
- net at R8.2: now also U1.11 (~{RESET}); no longer U1.14 (~{RESET})
- net VBUS: now reaches FB1.2, J1.A4 (VBUS), J1.A9 (VBUS), J1.B4 (VBUS), J1.B9 (VBUS)
- net VBUS: now also D5.5 (VBUS)

Commit message: layout
Parts:
- removed C7: 100nF, Cherry:C_0402_1005Metric, symbol Cherry:C
Changed lines of the file:
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@@
 	(wire
 		(pts
-			(xy 45.72 270.51) (xy 45.72 271.78)
-		)
-		(stroke
-			(width 0)
-			(type default)
-		)
-	)
-	(wire
-		(pts
 			(xy 259.08 58.42) (xy 261.62 58.42)
 		)
@@
 	(wire
 		(pts
-			(xy 45.72 262.89) (xy 45.72 261.62)
-		)
-		(stroke
-			(width 0)
-			(type default)
-		)
-	)
-	(wire
-		(pts
 			(xy 345.44 99.06) (xy 350.52 99.06)
 		)
@@
 	)
 	(symbol
-		(lib_id "Cherry:+3V3")
-		(at 45.72 261.62 0)
-		(unit 1)
-		(body_style 1)
-		(exclude_from_sim no)
-		(in_bom yes)
-		(on_board yes)
-		(in_pos_files yes)
-		(dnp no)
-		(property "Reference" "#PWR0562"
-			(at 45.72 259.08 0)
-			(hide yes)
-			(show_name no)
-			(do_not_autoplace no)
-			(effects
-				(font
-					(size 1.27 1.27)
-				)
-			)
-		)
-		(property "Value" "+3V3"
-			(at 45.72 257.53 0)
-			(show_name no)
-			(do_not_autoplace no)
-			(effects
-				(font
-					(size 1.27 1.27)
-				)
-			)
-		)
-		(property "Footprint" ""
-			(at 45.72 261.62 0)
-			(show_name no)
-			(do_not_autoplace no)
-			(effects
-				(font
-					(size 1.27 1.27)
-				)
-			)
-		)
-		(property "Datasheet" ""
-			(at 45.72 261.62 0)
-			(show_name no)
-			(do_not_autoplace no)
-			(effects
-				(font
-					(size 1.27 1.27)
-				)
-			)
-		)
-		(property "Description" ""
-			(at 45.72 261.62 0)
-			(show_name no)
-			(do_not_autoplace no)
-			(effects
-				(font
-					(size 1.27 1.27)
-				)
-			)
-		)
-		(pin "1"
-		)
-		(instances
-			(project "cherry"
-				(path "/00000000-0000-0000-0000-000000000001"
-					(reference "#PWR0562")
-					(unit 1)
-				)
-			)
-		)
-	)
-	(symbol
 		(lib_id "Cherry:GND")
 		(at 345.44 88.9 90)
@@
 	)
 	(symbol
-		(lib_id "Cherry:GND")
-		(at 45.72 271.78 0)
-		(unit 1)
-		(body_style 1)
-		(exclude_from_sim no)
-		(in_bom yes)
-		(on_board yes)
-		(in_pos_files yes)
-		(dnp no)
-		(property "Reference" "#PWR0564"
-			(at 45.72 269.24 0)
-			(hide yes)
-			(show_name no)
-			(do_not_autoplace no)
-			(effects
-				(font
-					(size 1.27 1.27)
-				)
-			)
-		)
-		(property "Value" "GND"
-			(at 45.72 275.87 0)
-			(show_name no)
-			(do_not_autoplace no)
-			(effects
-				(font
-					(size 1.27 1.27)
-				)
-			)
-		)
-		(property "Footprint" ""
-			(at 45.72 271.78 0)
-			(show_name no)
-			(do_not_autoplace no)
-			(effects
-				(font
-					(size 1.27 1.27)
-				)
-			)
-		)
-		(property "Datasheet" ""
-			(at 45.72 271.78 0)
-			(show_name no)
-			(do_not_autoplace no)
-			(effects
-				(font
-					(size 1.27 1.27)
-				)
-			)
-		)
-		(property "Description" ""
-			(at 45.72 271.78 0)
-			(show_name no)
-			(do_not_autoplace no)
-			(effects
-				(font
-					(size 1.27 1.27)
-				)
-			)
-		)
-		(pin "1"
-		)
-		(instances
-			(project "cherry"
-				(path "/00000000-0000-0000-0000-000000000001"
-					(reference "#PWR0564")
-					(unit 1)
-				)
-			)
-		)
-	)
-	(symbol
 		(lib_id "Cherry:+3V3")
 		(at 34.29 87.63 0)
@@
 					(unit 1)
 				)
-			)
-		)
-	)
-	(symbol
-		(lib_id "Cherry:C")
-		(at 45.72 266.7 0)
-		(unit 1)
-		(body_style 1)
-		(exclude_from_sim no)
-		(in_bom yes)
-		(on_board yes)
-		(in_pos_files yes)
-		(dnp no)
-		(property "Reference" "C7"
-			(at 49.17 265 0)
-			(show_name no)
-			(do_not_autoplace no)
-			(effects
-				(font
-					(size 1.27 1.27)
-				)
-			)
-		)
-		(property "Value" "100nF"
-			(at 50.745 268.4 0)
-			(show_name no)
-			(do_not_autoplace no)
-			(effects
-				(font
-					(size 1.27 1.27)
-				)
-			)
-		)
-		(property "Footprint" "Cherry:C_0402_1005Metric"
-			(at 45.72 266.7 0)
-			(hide yes)
-			(show_name no)
-			(do_not_autoplace no)
-			(effects
-				(font
-					(size 1.27 1.27)
-				)
-			)
-		)
-		(property "Datasheet" ""
-			(at 45.72 266.7 0)
-			(show_name no)
-			(do_not_autoplace no)
-			(effects
-				(font
-					(size 1.27 1.27)
-				)
-			)
-		)
-		(property "Description" ""
-			(at 45.72 266.7 0)
-			(show_name no)
-			(do_not_autoplace no)
-			(effects
-				(font
-					(size 1.27 1.27)
-				)
-			)
-		)
-		(pin "2"
-		)
-		(pin "1"
-		)
-		(instances
-			(project "cherry"
-				(path "/00000000-0000-0000-0000-000000000001"
-					(reference "C7")
-					(unit 1)
-				)

Commit message: refactor
Parts:
- R1: value 180k -> 100k
- R2: value 39.2k -> 22k
- U2: renamed from U3; value W25Q32JVSSIQ -> W25Q32JVSSIM; symbol Cherry:W25Q32JVSSIQ -> Cherry:W25Q32JVSSIM
- renumbered C11 to C10, C5 to C11, C13 to C12, C14 to C13, C15 to C14, C16 to C15, C17 to C16, C18 to C17, C19 to C18, C20 to C19, C21 to C20, C22 to C21, C23 to C22, C24 to C23, C25 to C24, C28 to C25, C6 to C5, C8 to C6, C9 to C7, C12 to C8, C10 to C9, J6 to J3, J3 to J4, J4 to J5, J5 to J6, R18 to R14, R19 to R15, R20 to R16, R21 to R17, R22 to R18, R14 to R19, R15 to R20, R16 to R21, R17 to R22, U2 to U3
Other:
- moved on the sheet: C10, C11, C12, C13, C14, C15, C16, C17, C18, C19, C20, C21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

Commit message: FT2232HL, 4-layer, renumber, pdf
Parts:
- added C17: 100nF, Cherry:C_0402_1005Metric, symbol Cherry:C
- C26: renamed from C11; value 4.7uF -> 10uF; footprint Cherry:C_0603_1608Metric -> Cherry:C_0805_2012Metric
- C27: footprint Cherry:C_0603_1608Metric -> Cherry:C_0805_2012Metric
- U1: value FT2232H-56Q -> FT2232HL; footprint Cherry:QFN-56-1EP_8x8mm_P0.5mm_EP5.9x5.9mm -> Cherry:LQFP-64_10x10mm_P0.5mm; symbol Cherry:FT2232H-56Q -> Cherry:FT2232HL
- renumbered C7 to C10, C8 to C11, C9 to C12, C10 to C13, C12 to C14, C13 to C15, C15 to C16, C16 to C18, C17 to C19, C19 to C20, C20 to C21, C21 to C22, C22 to C23, C23 to C24, C26 to C28, C14 to C5, C18 to C6, C24 to C7, C5 to C8, C6 to C9, R11 to R10, R12 to R11, R10 to R12
Connections:
- net +3V3: now also U1.20 (VCCIO), U1.31 (VCCIO), U1.42 (VCCIO), U1.56 (VCCIO), C17.1; no longer U1.16 (VCCIO), U1.36 (VCCIO), U1.44 (VREGIN)
- net +3V3A: now also U1.4 (VPHY); no longer U1.5 (VPHY)
- net CDONE: now also U1.23 (ADBUS6); no longer U1.19 (ADBUS6)
- net CLK_12M: now also U1.2 (OSCI); no longer U1.3 (OSCI)
- net FT_CRESET: now also U1.24 (ADBUS7); no longer U1.20 (ADBUS7)
- net FT_MISO: now also U1.18 (ADBUS2); no longer U1.14 (ADBUS2)
- net FT_MOSI: now also U1.17 (ADBUS1); no longer U1.13 (ADBUS1)
- net FT_SCK: now also U1.16 (ADBUS0); no longer U1.12 (ADBUS0)
- net FT_SS: now also U1.21 (ADBUS4); no longer U1.17 (ADBUS4)
- net GND: now also U1.1 (GND), U1.11 (GND), U1.13 (TEST), U1.15 (GND), U1.25 (GND), U1.35 (GND), U1.47 (GND), U1.5 (GND), U1.51 (GND), C17.2; no longer U1.21 (GND), U1.41 (GND), U1.45 (GND), U1.57 (GND)
- net UART_RX: now also U1.39 (BDBUS1); no longer U1.33 (BDBUS1)
- net UART_TX: now also U1.38 (BDBUS0); no longer U1.32 (BDBUS0)
- net VCORE: now also U1.12 (VCORE), U1.37 (VCORE), U1.49 (VREGOUT), U1.64 (VCORE); no longer U1.2 (VCORE), U1.31 (VCORE), U1.43 (VREGOUT)
- net at R8.2: now also U1.14 (~{RESET}); no longer U1.11 (~{RESET})
