File: cherry/pcb/src/cherry.kicad_sch (KiCad schematic)
At the start: 73 parts, among them J1 USB4085-GF-A, J2 PinHeader_1x24, J3 PinHeader_1x24, J4 PinHeader_1x06, J5 PinHeader_1x06, J6 PinHeader_1x06, SW1 RESET, SW2 USER, U1 FT2232HL, U2 W25Q32JVSSIM, U3 ICE40LP8K-CM81, U4 TPS62A02, U5 TPS62A02, X1 ASE-12.000MHZ-LR-T

Commit message: wip
Parts:
- removed C12, C13, C14, C15: 100nF, Cherry:C_0402_1005Metric, symbol Cherry:C
- removed C26, C5: 10uF, Cherry:C_0805_2012Metric, symbol Cherry:C
- removed FB2: BLM21AG601SH1D, Cherry:L_0805_2012Metric, symbol Cherry:Ferrite_Bead
- removed J4, J6: PinHeader_1x06, Cherry:PinHeader_1x06_P2.54mm, symbol Cherry:PinHeader_1x06
- removed R18: 1k, Cherry:R_0402_1005Metric, symbol Cherry:R
- removed R7: 12k, Cherry:R_0402_1005Metric, symbol Cherry:R
- removed SW2: USER, Cherry:SW_Push_1P1T_NO_CK_KMR2, symbol Cherry:SW_Push
- removed U1: FT2232HL, Cherry:LQFP-64_10x10mm_P0.5mm, symbol Cherry:FT2232HL
- added C29: 100nF, Cherry:C_0402_1005Metric, symbol Cherry:C
- added D6: LED_AMBER_0603, Cherry:LED_0603_1608Metric, symbol Cherry:LED
- added Q1: BSS138, Package_TO_SOT_SMD:SOT-23, symbol Transistor_FET:Q_NMOS_GSD
- added R23, R24, R27: 10k, Cherry:R_0402_1005Metric, symbol Cherry:R
- added R25, R26, R29: 1k, Cherry:R_0402_1005Metric, symbol Cherry:R
- added SW2: IMAGE SELECT, Button_Switch_SMD:SW_DIP_SPSTx02_Slide_Copal_CHS-02A_W5.08mm_P1.27mm_JPin, symbol Switch:SW_DIP_x02
- added SW3: USER, Cherry:SW_Tactile_XKB_TS-1187A, symbol Cherry:SW_Push
- C1, C2, C27, C6, C7: LCSC (none) -> C15850
- C10, C11, C16, C17, C18, C19, C20, C21, C22, C23, C24, C25, C28, C8, C9: LCSC (none) -> C1525
- C3, C4: LCSC (none) -> C45783
- D1: value PWR -> KT-0603R; LCSC (none) -> C2286
- D2: value CFG -> KT-0603R; LCSC (none) -> C2286
- D3: value USER0 -> KT-0603R; LCSC (none) -> C2286
- D4: value USER1 -> KT-0603R; LCSC (none) -> C2286
- D5: LCSC (none) -> C2687116
- FB1: value BLM21AG601SH1D -> GZ2012D601TF; LCSC (none) -> C1017
- J1: value USB4085-GF-A -> TYPE-C-31-M-12; footprint Cherry:USB_C_Receptacle_GCT_USB4085 -> Cherry:USB_C_Receptacle_Hroparts_TYPE-C-31-M-12; LCSC (none) -> C165948
- J2, J3: value PinHeader_1x24 -> PinHeader_2x24_Duplicate; footprint Cherry:PinHeader_1x24_P2.54mm -> Cherry:PinHeader_2x24_P2.54mm_Duplicate; now not fitted
- J5: value PinHeader_1x06 -> SPI PROGRAM; now not fitted
- L1, L2: value 1uH -> TFM201208ALD-1R0MTCA; footprint Cherry:L_0805_2012Metric -> Cherry:L_TDK_TFM201208ALD; LCSC (none) -> C433051
- R1, R3, R4: LCSC (none) -> C25741
- R10, R11, R8: LCSC (none) -> C25744
- R12, R19, R20, R21, R22: LCSC (none) -> C11702
- R13: LCSC (none) -> C25076
- R14, R15: value 470 -> 68; LCSC (none) -> C25117
- R16: value 470 -> 1.5k; LCSC (none) -> C25117
- R17: value 470 -> 10k; LCSC (none) -> C25744
- R2: LCSC (none) -> C25768
- R5, R6: LCSC (none) -> C25905
- R9: value 10k -> 100k; LCSC (none) -> C25741
- SW1: value RESET -> TS-1187A-B-A-B; footprint Cherry:SW_Push_1P1T_NO_CK_KMR2 -> Cherry:SW_Tactile_XKB_TS-1187A; LCSC (none) -> C318884
- U2: value W25Q32JVSSIM -> W25Q32JVSSIQ; LCSC (none) -> C179173
- U3: value ICE40LP8K-CM81 -> ICE40HX8K-BG121; footprint Cherry:BGA-81_9x9_8.0x8.0mm_P0.8mm -> Package_BGA:BGA-121_9.0x9.0mm_Layout11x11_P0.8mm_Ball0.4mm_Pad0.35mm_NSMD; symbol Cherry:ICE40LP8K-CM81 -> Cherry:ICE40HX8K-BG121
- U4, U5: value TPS62A02 -> TPS62A02APDDCR; LCSC (none) -> C25687169
- X1: value ASE-12.000MHZ-LR-T -> OXETDLJANF-48.000000MHz; footprint Cherry:Oscillator_SMD_Abracon_ASE-4Pin_3.2x2.5mm -> Cherry:Oscillator_SMD_Taitien_OX_3.2x2.5mm; LCSC (none) -> C5173414
Connections:
- net FT_SS is gone; now on net CRESET_B: R17.1
- net GPIO_38 is gone; now on net LED1: U3.J3 (IOB_57)
- net GPIO_39 is gone; now on net +1V2: U3.H4 (VCC)
- net GPIO_40 is gone; now on net GND: U3.G5 (GND)
- net GPIO_41 is gone; now on net GND: U3.H5 (GND)
- net GPIO_52 is gone; now on net +1V2: U3.D8 (VCC)
- net UART_TX is gone; now on net QSPI_IO3: U3.J8 (IOB_91)
- net +1V2: now also U3.H8 (VCC); no longer U3.E9 (VCC), U3.F2 (VCC)
- net +3V3: now also R17.2, R20.1, U3.C10 (VPP_2V5), U3.D6 (VCCIO_0), U3.E4 (VCCIO_3), U3.F8 (VCCIO_1), U3.G4 (VCCIO_3), U3.H6 (VCCIO_2), U3.L11 (VCC_SPI), R27.1, SW2.3, SW2.4; no longer R9.1, U2.3 (~{WP}), U2.7 (~{HOLD}), U3.A5 (VCCIO_0), U3.C6 (VCCIO_1), U3.C8 (VPP_2V5), U3.H3 (VCCIO_3), U3.H8 (VCC_SPI), U3.J5 (VCCIO_2)
- net +5V: now also R9.1; no longer U4.1 (EN), U5.1 (EN)
- net CDONE: now also U3.K8 (CDONE), Q1.1 (G); no longer R20.1, U3.E6 (CDONE)
- net CRESET_B: now also J5.2 (Pin_2), U3.L9 (~{CRESET}); no longer R9.2, SW1.1, U3.H6 (CRESET_B)
- net GND: now also J5.1 (Pin_1), U3.E5 (GND), U3.E6 (GND), U3.E7 (GND), U3.F7 (GND), U3.G6 (GND), U3.G7 (GND), C29.2, D6.1 (K), Q1.2 (S), R23.2, R24.2, SW3.2; no longer D2.1 (K), U3.F4 (GND), U3.F9 (GND)
- net GNDPLL: now also U3.C5 (GNDPLL1), U3.L6 (GNDPLL0); no longer U3.J6 (GNDPLL0)
- net GPIO_12: now also U3.A5 (IOT_207); no longer U3.E4 (IOL_14B)
- net GPIO_26: now also U3.C7 (IOT_191); no longer U3.C5 (IOT_197_GBIN1)
- net GPIO_30: now also U3.C8 (IOT_179); no longer U3.E5 (IOT_214)
- net LED1: no longer U3.J9 (IOR_110)
- net USB_DM: no longer D5.6 (I/O1)
- net USB_DP: no longer D5.4 (I/O2)
- net VCCPLL: now also U3.C6 (VCCPLL1), U3.J6 (VCCPLL0); no longer U3.J7 (VCCPLL0)
- net QSPI_IO2: now reaches R8.2
- net QSPI_IO2: now also U2.3 (~{WP}), U3.K6 (IOB_82_GBIN4)
- net BTN renamed QSPI_IO3
- net QSPI_IO3: now also U2.7 (~{HOLD}); no longer U3.C4 (IOT_198_GBIN0)
- net CLK_12M renamed CLK_48M
- net CLK_48M: now also U3.E10 (IOR_141_GBIN2); no longer U3.G4 (IOB_81_GBIN5)
- net FT_MISO renamed USB_PULLUP
- net USB_PULLUP: now also U3.A3 (IOT_223)
- net FT_MOSI renamed USB_DM_ESD
- net USB_DM_ESD: now also D5.6 (I/O1)
- net FT_SCK renamed USB_DP_ESD
- net USB_DP_ESD: now also D5.4 (I/O2)
- net GPIO_27: no longer names the net of J3.9
- net GPIO_27: no longer U3.A4 (IOT_208)
- net GPIO_28: no longer names the net of J3.10
- net GPIO_28: no longer U3.B4 (IOT_211)
- net GPIO_31: no longer names the net of J3.13
- net GPIO_31: no longer U3.A3 (IOT_217)
- net GPIO_37: no longer names the net of U3.J2 (IOL_25B)
- net GPIO_42: no longer names the net of U3.G9 (IOR_128)
- removed net GPIO_43: J5.1 (Pin_1), U3.F8 (IOR_113)
- net GPIO_44: no longer names the net of U3.G8 (IOR_118)
- net GPIO_44: no longer J5.2 (Pin_2)
- net GPIO_45 renamed QSPI_CS_B
- net QSPI_CS_B: now also R10.2, U2.1 (~{CS}), U3.K10 (IOB_108_SS); no longer U3.D6 (IOR_115)
- net GPIO_46: no longer names the net of U3.A9 (IOT_178)
- net GPIO_46: no longer J5.4 (Pin_4)
- net GPIO_47: no longer names the net of U3.D7 (IOT_181)
- net GPIO_47: no longer J5.5 (Pin_5)
- net GPIO_48 renamed QSPI_IO1
- net QSPI_IO1: now also U2.2 (DO), U3.J9 (IOB_106_SDI); no longer U3.E7 (IOR_118)
- net GPIO_49: no longer names the net of U3.D9 (IOR_147)
- net GPIO_50: no longer names the net of U3.B9 (IOT_174)
- net GPIO_51: no longer names the net of U3.E8 (IOR_146)
- net GPIO_53: no longer names the net of U3.C9 (IOT_172)
- removed net SPI_MISO: R16.2, U2.2 (DO), U3.H7 (IOB_106_SDI)
- removed net SPI_MOSI: R15.2, U2.5 (DI), U3.G6 (IOB_105_SDO)
- removed net SPI_SCK: R14.2, U2.6 (CLK), U3.G7 (IOB_107_SCK)
- removed net SPI_SS: R10.2, R17.2, U2.1 (~{CS}), U3.F7 (IOB_108_SS)
- net UART_RX renamed CBSEL1
- net CBSEL1: now also R24.1, R26.1
- new net: R25.2, SW2.1
- new net: R26.2, SW2.2
- new net: U3.D11 (IOR_152), U3.E11 (IOR_148), U3.E9 (IOR_144), U3.F10 (IOR_136), U3.F11 (IOR_140_GBIN3), U3.F2 (IOL_12B), U3.F4 (IOL_13A), U3.F9 (IOR_137), U3.G10 (IOR_120), U3.G11 (IOR_129), U3.H10 (IOR_116), U3.H11 (IOR_119), U3.H3 (IOL_17B), U3.H7 (IOB_87), U3.J11 (IOR_114), U3.J5 (IOB_78), U3.J7 (IOB_86), U3.K1 (IOL_23B), U3.K11 (IOR_115), U3.K2 (IOL_25A), U3.K3 (IOB_63), U3.K4 (IOB_73), U3.K5 (IOB_79), U3.K7 (IOB_89), U3.L1 (IOB_56), U3.L2 (IOB_61), U3.L3 (IOB_71), U3.L4 (IOB_72), U3.L5 (IOB_81_GBIN5), U3.L7 (IOB_94)
- new net: D6.2 (A), R29.2
- new net CBSEL0: R23.1, R25.1, U3.L8 (IOB_103_CBSEL0)
- new net CFG_LED_K: D2.1 (K), Q1.3 (D)
- new net PROG_LED: R29.1, U3.J10 (IOR_117)
- new net PWR_EN: C29.1, R9.2, SW1.1, U4.1 (EN), U5.1 (EN)
- new net QSPI_IO0: J5.5 (Pin_5), U2.5 (DI), U3.K9 (IOB_105_SDO)
- new net QSPI_SCK: J5.4 (Pin_4), U2.6 (CLK), U3.L10 (IOB_107_SCK)
- new net USB_DM_FPGA: R15.2, U3.A4 (IOT_211)
- new net USB_DP_FPGA: R14.2, R16.2, U3.B4 (IOT_219)
- new net USER_BTN: R27.2, SW3.1, U3.C4 (IOL_4A)
- no-connect marks 35 -> 22
Other:
- note added: "48MHz Clock"
- note added: "IMAGE 1:0 (ON = 1)"
- note added: "MODE / PROG"
- note added: "Native USB - FPGA Full Speed"
- note added: "Quad SPI Flash"
- note added: "RESET (rail power-cycle)"
- note removed: "12MHz Clock"
- note removed: "Decoupling - FT2232H"
- note removed: "SPI Flash"
- note removed: "USB Bridge - FT2232HL"
