File: boards/cherry/pcb/src/cherry.kicad_sch (KiCad schematic)
At the start: 71 parts, among them J1 TYPE-C-31-M-12, J2 PinHeader_2x24_Duplicate, J3 PinHeader_2x24_Duplicate, J5 SPI PROGRAM, Q1 BSS138, SW1 TS-1187A-B-A-B, SW2 IMAGE SELECT, SW3 USER, U2 W25Q32JVSSIQ, U3 ICE40HX8K-BG121, U4 TPS62A02APDDCR, U5 TPS62A02APDDCR, X1 OXETDLJANF-48.000000MHz

Commit message: wip
Parts:
- removed D2: KT-0603R, Cherry:LED_0603_1608Metric, symbol Cherry:LED
- removed Q1: BSS138, Package_TO_SOT_SMD:SOT-23, symbol Transistor_FET:Q_NMOS_GSD
- removed R20: 1k, Cherry:R_0402_1005Metric, symbol Cherry:R
- removed SW2: IMAGE SELECT, Button_Switch_SMD:SW_DIP_SPSTx02_Slide_Copal_CHS-02A_W5.08mm_P1.27mm_JPin, symbol Switch:SW_DIP_x02
- added JP1: IMAGE0, Jumper:SolderJumper-2_P1.3mm_Open_RoundedPad1.0x1.5mm, symbol Jumper:SolderJumper_2_Open
- added JP2: IMAGE1, Jumper:SolderJumper-2_P1.3mm_Open_RoundedPad1.0x1.5mm, symbol Jumper:SolderJumper_2_Open
Connections:
- net +3V3: now also JP1.2 (B), JP2.2 (B)
- net GPIO_28: now reaches J3.10
- net GPIO_28: now also U3.B9 (IOT_174)
- net GPIO_31: now reaches J3.13
- net GPIO_31: now also U3.C9 (IOT_172)
- net GPIO_27: now reaches J3.9
- net GPIO_27: now also U3.A9 (IOT_178)
- net at R25.2: now also JP1.1 (A)
- net at R26.2: now also JP2.1 (A)
- no-connect marks 22 -> 16
Other:
- note added: "IMAGE 1:0 (BRIDGE = 1)"
- note removed: "IMAGE 1:0 (ON = 1)"
