File: boards/cherry/pcb/src/cherry.kicad_pcb (KiCad board)
At the start: 4 copper layers, 61.2 x 31.2 mm, 71 parts, among them J1 TYPE-C-31-M-12, J2 PinHeader_2x24_Duplicate, J3 PinHeader_2x24_Duplicate, J5 SPI PROGRAM, Q1 BSS138, SW1 TS-1187A-B-A-B, SW2 IMAGE SELECT, SW3 USER, U2 W25Q32JVSSIQ, U3 ICE40HX8K-BG121, U4 TPS62A02APDDCR, U5 TPS62A02APDDCR, X1 OXETDLJANF-48.000000MHz

Commit message: wip
Parts:
- removed D2: KT-0603R, Cherry:LED_0603_1608Metric
- removed Q1: BSS138, Package_TO_SOT_SMD:SOT-23
- removed R20: 1k, Cherry:R_0402_1005Metric
- removed SW2: IMAGE SELECT, Button_Switch_SMD:SW_DIP_SPSTx02_Slide_Copal_CHS-02A_W5.08mm_P1.27mm_JPin
- added JP1: IMAGE0, Jumper:SolderJumper-2_P1.3mm_Open_RoundedPad1.0x1.5mm, F.Cu at (146.7, 93.4)
- added JP2: IMAGE1, Jumper:SolderJumper-2_P1.3mm_Open_RoundedPad1.0x1.5mm, F.Cu at (146.7, 96.1)
Connections:
- J3 pad 10: unconnected-(J3-Pad10) -> /GPIO_28
- J3 pad 13: unconnected-(J3-Pad13) -> /GPIO_31
- J3 pad 9: unconnected-(J3-Pad9) -> /GPIO_27
- U3 pad A9: unconnected-(U3-IOT_178-PadA9) -> /GPIO_27
- U3 pad B9: unconnected-(U3-IOT_174-PadB9) -> /GPIO_28
- U3 pad C9: unconnected-(U3-IOT_172-PadC9) -> /GPIO_31

Commit message: wip
Parts:
- moved R25 5.77 mm to (144.1, 83.8)
- moved C9 3.50 mm to (137.7, 86.1), turned to 90 degrees
- moved U2 1.50 mm to (141.2, 90.2)
Changed lines of the file:
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@@
 	(footprint "Cherry:SOIC-8_5.3x5.3mm_P1.27mm"
 		(layer "F.Cu")
-		(at 139.7 90.17 90)
+		(at 141.2 90.17 90)
 		(descr "SOIC, 8 Pin (JEITA/EIAJ ED-7311-19 variation 08-001-BBA and Atmel/Microchip, 208 mils width, https://www.jeita.or.jp/japanese/standard/book/ED-7311-19/#target/page_no=21, https://ww1.microchip.com/downloads/en/DeviceDoc/20005045C.pdf#page=23, https://ww1.microchip.com/downloads/en/DeviceDoc/doc2535.pdf#page=162)")
 		(tags "SOIC SO P-SOP SOP SOP-8 SO SO-8 8S2 S2AE/F K04-056 CASE-751BE SO8W 8-Pin-SOIC PSA W8-2 W8-4 W8MS-1 FPT-8P-M08")
@@
 	(footprint "Cherry:R_0402_1005Metric"
 		(layer "F.Cu")
-		(at 144.145 89.59 90)
+		(at 144.145 83.82 90)
 		(descr "Resistor SMD 0402 (1005 Metric), square (rectangular) end terminal, IPC-7351 nominal, (Body size source: IPC-SM-782 page 72, https://www.pcb-3d.com/wordpress/wp-content/uploads/ipc-sm-782a_amendment_1_and_2.pdf)")
 		(tags "resistor")
@@
 	(footprint "Cherry:C_0402_1005Metric"
 		(layer "F.Cu")
-		(at 135 83.82)
+		(at 137.65 86.1025 90)
 		(descr "Capacitor SMD 0402 (1005 Metric), square (rectangular) end terminal, IPC-7351 nominal, (Body size source: IPC-SM-782 page 76, https://www.pcb-3d.com/wordpress/wp-content/uploads/ipc-sm-782a_amendment_1_and_2.pdf)")
 		(tags "capacitor")
