File: boards/grape/pcb/src/grape.kicad_pcb (KiCad board)
At the start: 4 copper layers, 84 x 64 mm, 136 parts, among them J1 USB-C USB2 Device, J2 GPIO 0-27, J3 GPIO 28-55, J4 JTAG, Q1 BSS138, SW1 IMAGE[1:0], SW2 COLD RESET, SW3 PROGRAM, U1 XC7A35T-1FTG256C, U2 TPS62A02DRL, U3 TPS62A02DRL, U4 TPS62A02DRL, U5 W25Q128JVSIQ, U6 USBLC6-2SC6, U7 TPS22917DBV, X1 ASE-48.000MHz

Commit message: wip
Parts:
- C22: moved to B.Cu
- moved C21 1.41 mm to (50.0, 53.5)
- moved C22 1.12 mm to (50.0, 58.0)
- moved C36 0.64 mm to (73.2, 39.0)
- moved R40 0.50 mm to (76.5, 48.0)
- moved R41 0.50 mm to (76.5, 50.5)
- moved R42 0.50 mm to (76.5, 53.0)
- moved R43 0.50 mm to (76.5, 55.5)
- moved R44 0.50 mm to (76.5, 58.0)
- moved R45 0.50 mm to (76.5, 60.5)
