File: boards/cherry/board/src/cherry.kicad_pcb (KiCad board)
At the start: 4 copper layers, 61.2 x 31.2 mm, 69 parts, among them J1 TYPE-C-31-M-12, J2 PinHeader_2x24_Duplicate, J3 PinHeader_2x24_Duplicate, J5 SPI PROGRAM, SW1 TS-1187A-B-A-B, SW3 USER, U2 W25Q32JVSSIQ, U3 ICE40HX8K-BG121, U4 TPS62A02APDDCR, U5 TPS62A02APDDCR, X1 OXETDLJANF-48.000000MHz

Commit message: wip
Parts:
- removed JP2: IMAGE1, Jumper:SolderJumper-2_P1.3mm_Open_RoundedPad1.0x1.5mm
- removed R26: 1k, Cherry:R_0402_1005Metric
- JP1: value IMAGE0 -> USER; moved to B.Cu
- moved D1 45.9 mm to (148.6, 86.4), turned to 180 degrees
- moved R19 42.6 mm to (148.6, 83.8), turned to 90 degrees
- moved R9 32.4 mm to (149.9, 83.8)
- moved C29 23.9 mm to (142.2, 83.8), turned to -90 degrees
- moved R24 13.4 mm to (134.6, 88.3), turned to 0 degrees
- moved R12 13.1 mm to (120.0, 94.0), turned to 0 degrees
- moved R23 12.7 mm to (134.6, 85.7), turned to 0 degrees
- moved JP1 12.5 mm to (134.6, 90.2), turned to -90 degrees
- moved R11 10.5 mm to (134.6, 93.3), turned to 180 degrees
- moved R25 10.0 mm to (134.6, 87.0), turned to 0 degrees
- moved R22 8.98 mm to (147.3, 96.5), turned to -90 degrees
- moved D3 8.35 mm to (148.6, 88.9)
- moved D6 8.35 mm to (148.6, 94.0)
- moved D4 8.35 mm to (148.6, 91.4)
- moved R13 7.96 mm to (134.6, 89.5), turned to 180 degrees
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- renumbered J5 to J4, SW3 to SW2
Connections:
- D1 pad 1: GND -> Net-(D1-K)
- D1 pad 2: Net-(D1-A) -> +3V3
- D3 pad 1: GND -> Net-(D3-K)
- D3 pad 2: Net-(D3-A) -> /LED0
- D4 pad 1: GND -> Net-(D4-K)
- D4 pad 2: Net-(D4-A) -> /LED1
- D5 pad 1: /USB_DM -> /USB_DP
- D5 pad 3: /USB_DP -> /USB_DM
- D5 pad 4: /USB_DP_ESD -> /USB_DM_ESD
- D5 pad 6: /USB_DM_ESD -> /USB_DP_ESD
- D6 pad 1: GND -> Net-(D6-K)
- D6 pad 2: Net-(D6-A) -> /PROG_LED
- R10 pad 2: /QSPI_CS_B -> /QSPI_SS
- R16 pad 1: /USB_PULLUP -> /USB_PU_FPGA
- R16 pad 2: /USB_DP_FPGA -> /USB_DP_ESD
- R19 pad 1: +3V3 -> Net-(D1-K)
- R19 pad 2: Net-(D1-A) -> GND
- R21 pad 1: /LED0 -> Net-(D3-K)
- R21 pad 2: Net-(D3-A) -> GND
- R22 pad 1: /LED1 -> Net-(D4-K)
- R22 pad 2: Net-(D4-A) -> GND
- R29 pad 1: /PROG_LED -> Net-(D6-K)
- R29 pad 2: Net-(D6-A) -> GND
- U2 pad 1: /QSPI_CS_B -> /QSPI_SS
- U3 pad K10: /QSPI_CS_B -> /QSPI_SS
Other:
- board text removed: "0"
- board text removed: "1"
- board text removed: "IMAGE"
- board text removed: "PROG"
- board text removed: "SPI >"
- board text removed: "USR"

Commit message: r
Parts:
- J2, J3: value PinHeader_2x24_Duplicate -> PinHeader_2x24
- R9: value 100k -> 10k
Connections:
- net /QSPI_CS_B renamed /QSPI_CS
- net /USB_DM renamed /USB_DM_PIN
- net /USB_DP renamed /USB_DP_PIN
- D3 pad 2: /LED0 -> unconnected-(D3-A-Pad2)
- D4 pad 2: /LED1 -> unconnected-(D4-A-Pad2)
- D5 pad 5: /VBUS -> +5V
- D6 pad 2: /PROG_LED -> unconnected-(D6-A-Pad2)
- FB1 pad 2: /VBUS -> Net-(FB1-Pad2)
- J1 pad A4: /VBUS -> Net-(FB1-Pad2)
- J1 pad A9: /VBUS -> Net-(FB1-Pad2)
- J1 pad B4: /VBUS -> Net-(FB1-Pad2)
- J1 pad B9: /VBUS -> Net-(FB1-Pad2)
- J2 pad 6: /CRESET_B -> /CRESET
- J4 pad 2: /CRESET_B -> /CRESET
- JP1 pad 1: Net-(JP1-A) -> /CBSEL0
- R16 pad 1: /USB_PU_FPGA -> /USB_DP_ESD
- R16 pad 2: /USB_DP_ESD -> /USB_PU_FPGA
- R17 pad 1: /CRESET_B -> +3V3
- R17 pad 2: +3V3 -> /CRESET
- U3 pad L9: /CRESET_B -> /CRESET

Commit message: wip
Parts:
- added JP2: USER, Cherry:SolderJumper-2_P1.3mm_Open_RoundedPad1.0x1.5mm, B.Cu at (165.1, 92.7)
- J2, J3: value PinHeader_2x24 -> Conn_02x24_Odd_Even; footprint Cherry:PinHeader_2x24_P2.54mm_Duplicate -> Connector_PinHeader_2.54mm:PinHeader_2x24_P2.54mm_Vertical
- J4: footprint Cherry:PinHeader_1x06_P2.54mm -> Connector_PinHeader_2.54mm:PinHeader_1x06_P2.54mm_Vertical
- JP1: footprint Jumper:SolderJumper-2_P1.3mm_Open_RoundedPad1.0x1.5mm -> Cherry:SolderJumper-2_P1.3mm_Open_RoundedPad1.0x1.5mm
- moved JP1 30.9 mm to (165.1, 95.2), turned to 180 degrees
- moved R10 14.9 mm to (109.2, 97.8), turned to 90 degrees
- moved R13 12.1 mm to (123.8, 87.6), turned to 0 degrees
- moved R12 9.55 mm to (123.8, 86.4)
- moved U3 7.24 mm to (113.7, 90.2), turned to 180 degrees
- moved R5 5.85 mm to (123.8, 92.7)
- moved D1 4.62 mm to (113.7, 85.7)
- moved R11 4.49 mm to (110.5, 97.8), turned to 90 degrees
- moved R14 4.12 mm to (113.0, 97.8), turned to 90 degrees
- moved U2 4.12 mm to (131.1, 90.2), turned to 0 degrees
- moved R16 4.02 mm to (146.1, 97.8)
- moved R20 4.02 mm to (143.5, 97.8)
- moved R21 4.02 mm to (144.8, 97.8)
- moved R15 4.02 mm to (146.1, 82.5)
- moved R18 4.02 mm to (144.8, 82.5)
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- renumbered C27 to C1, C16 to C12, C17 to C13, C6 to C14, C18 to C15, C19 to C16, C7 to C17, C20 to C18, C21 to C19, C28 to C2, C22 to C20, C23 to C21, C24 to C22, C25 to C23, C1 to C3, C3 to C4, C2 to C5, C4 to C6, C29 to C7, D5 to D1, D1 to D2, D6 to D5, R13 to R1, R5 to R10, R6 to R11, R1 to R12, R2 to R13, R3 to R14, R9 to R15, R27 to R16, R4 to R17, R19 to R18, R21 to R19, R10 to R2, R22 to R20, R29 to R21, R23 to R22, R24 to R23, R8 to R3, R11 to R4, R17 to R5, R12 to R6, R14 to R7, R15 to R8, R16 to R9, U2 to U1, U3 to U2, U4 to U3, U5 to U4
Connections:
- net /PWR_EN renamed /PWRSW
- net /USB_DM_ESD renamed /USB_ESD_DM
- net /USB_DM_FPGA renamed /USB_DM
- net /USB_DM_PIN renamed /USB_PIN_DM
- net /USB_DP_ESD renamed /USB_ESD_DP
- net /USB_DP_FPGA renamed /USB_DP
- net /USB_DP_PIN renamed /USB_PIN_DP
- net /USER_BTN renamed /BTN
- net Net-(FB1-Pad2) renamed /VBUD
- net Net-(J1-CC1) renamed /CC1
- net Net-(J1-CC2) renamed /CC2
- net Net-(U4-FB) renamed /FB3V3
- net Net-(U5-FB) renamed /FB1V2
- D3 pad 2: unconnected-(D3-A-Pad2) -> /PROG
- D4 pad 2: unconnected-(D4-A-Pad2) -> /LED1
- D5 pad 2: unconnected-(D6-A-Pad2) -> /LED2
- J2 pad 10: /GPIO_4 -> /GPIO_33
- J2 pad 11: /GPIO_5 -> /GPIO_2
- J2 pad 12: /GPIO_6 -> /GPIO_34
- J2 pad 13: /GPIO_7 -> /GPIO_3
- J2 pad 14: /GPIO_8 -> /GPIO_35
- J2 pad 15: /GPIO_9 -> /GPIO_4
- J2 pad 16: /GPIO_10 -> /GPIO_36
- J2 pad 17: /GPIO_11 -> GND
- J2 pad 18: /GPIO_12 -> +3V3
- J2 pad 19: /GPIO_13 -> /GPIO_5
- J2 pad 2: +3V3 -> +5V
- J2 pad 20: /GPIO_14 -> /GPIO_37
- J2 pad 21: /GPIO_15 -> /GPIO_6
- J2 pad 22: /GPIO_16 -> /GPIO_38
- J2 pad 23: /GPIO_17 -> /GPIO_7
- J2 pad 24: /GPIO_18 -> /GPIO_39
- J2 pad 3: GND -> +3V3
- J2 pad 4: GND -> +3V3
- J2 pad 5: GND -> /CRESET
- J2 pad 6: /CRESET -> unconnected-(J2-Pin_6-Pad6)
- J2 pad 7: /GPIO_1 -> GND
- J2 pad 8: /GPIO_2 -> +3V3
- J2 pad 9: /GPIO_3 -> /GPIO_1
- J3 pad 1: /GPIO_19 -> GND
- J3 pad 10: /GPIO_28 -> /GPIO_52
- J3 pad 11: /GPIO_29 -> GND
- J3 pad 12: /GPIO_30 -> +3V3
- J3 pad 13: /GPIO_31 -> /GPIO_21
- J3 pad 14: /GPIO_32 -> /GPIO_53
- J3 pad 15: /GPIO_33 -> /GPIO_22
- J3 pad 16: /GPIO_34 -> /GPIO_54
- J3 pad 17: /GPIO_35 -> /GPIO_23
- J3 pad 18: /GPIO_36 -> /GPIO_55
- J3 pad 19: GND -> /GPIO_24
- J3 pad 2: /GPIO_20 -> +3V3
- J3 pad 20: GND -> /GPIO_56
- J3 pad 22: GND -> +3V3
- J3 pad 23: +3V3 -> /GPIO_25
- J3 pad 24: +5V -> /GPIO_57
- J3 pad 3: /GPIO_21 -> /GPIO_17
- J3 pad 4: /GPIO_22 -> /GPIO_49
- J3 pad 5: /GPIO_23 -> /GPIO_18
- J3 pad 6: /GPIO_24 -> /GPIO_50
- J3 pad 7: /GPIO_25 -> /GPIO_19
- J3 pad 8: /GPIO_26 -> /GPIO_51
- J3 pad 9: /GPIO_27 -> /GPIO_20
- R9 pad 2: /USB_PU_FPGA -> /USB_PU
- U2 pad A3: /USB_PULLUP -> /USB_PU
- U2 pad J10: /PROG_LED -> /PROG
- U2 pad J3: /LED1 -> /LED2
- U2 pad J4: /LED0 -> /LED1
Other:
- board text added: "BTN"
- board text added: "LED0"
- board text added: "LED1"
- board text added: "PROG"
- board text added: "PWR"

Commit message: chore
Parts:
- added C24: 100nF, Cherry:C_0402_1005Metric, F.Cu at (146.7, 91.4)
- added D6: KT-0603R, Cherry:LED_0603_1608Metric, F.Cu at (149.9, 94.0)
- added D7: KT-0603R, Cherry:LED_0603_1608Metric, F.Cu at (149.9, 96.5)
- added R24: 1k, Cherry:R_0402_1005Metric, F.Cu at (146.7, 88.9)
- J2, J3, J4: moved to F.Cu
- R14: renamed from R6; value 1k -> 10k
- moved R3 16.6 mm to (111.8, 97.8), turned to 90 degrees
- moved R4 14.8 mm to (113.0, 97.8), turned to -90 degrees
- moved JP1 13.3 mm to (152.4, 91.4)
- moved JP2 13.3 mm to (152.4, 88.9)
- moved R15 9.09 mm to (134.6, 97.2), turned to 90 degrees
- moved R25 9.09 mm to (146.7, 90.2)
- moved R19 5.99 mm to (146.7, 87.6), turned to 180 degrees
- moved R12 5.85 mm to (142.2, 97.2), turned to 90 degrees
- moved C2 5.43 mm to (133.3, 97.2), turned to -90 degrees
- moved R21 5.43 mm to (146.7, 92.7), turned to 0 degrees
- moved R20 4.96 mm to (146.7, 94.0), turned to 0 degrees
- moved D5 4.62 mm to (149.9, 91.4)
- moved R18 4.26 mm to (146.7, 86.4), turned to 180 degrees
- moved R22 3.86 mm to (142.2, 83.2)
- moved R7 3.86 mm to (123.2, 87.6)
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- renumbered R10 to R1, R2 to R10, R3 to R11, R4 to R12, R5 to R13, R1 to R15, R22 to R16, R23 to R17, R11 to R2, R15 to R22, R16 to R23, R12 to R3, R13 to R4, R14 to R5, R17 to R6, R9 to R7, R7 to R8, R8 to R9
Connections:
- net /VBUD renamed /VBUS
- C1 pad 2: /GNDPLL -> GND
- C2 pad 2: /GNDPLL -> GND
- D4 pad 2: /LED1 -> /LED0
- D5 pad 2: /LED2 -> /LED1
- J2 pad 10: /GPIO_33 -> /GPIO_5
- J2 pad 12: /GPIO_34 -> /GPIO_6
- J2 pad 14: /GPIO_35 -> /GPIO_7
- J2 pad 16: /GPIO_36 -> /GPIO_8
- J2 pad 19: /GPIO_5 -> /GPIO_9
- J2 pad 20: /GPIO_37 -> /GPIO_13
- J2 pad 21: /GPIO_6 -> /GPIO_10
- J2 pad 22: /GPIO_38 -> /GPIO_14
- J2 pad 23: /GPIO_7 -> /GPIO_11
- J2 pad 24: /GPIO_39 -> /GPIO_15
- J2 pad 25: /GPIO_8 -> /GPIO_12
- J2 pad 26: /GPIO_40 -> /GPIO_16
- J2 pad 29: /GPIO_9 -> /GPIO_17
- J2 pad 30: /GPIO_41 -> /GPIO_21
- J2 pad 31: /GPIO_10 -> /GPIO_18
- J2 pad 32: /GPIO_42 -> /GPIO_22
- J2 pad 33: /GPIO_11 -> /GPIO_19
- J2 pad 34: /GPIO_43 -> /GPIO_23
- J2 pad 35: /GPIO_12 -> /GPIO_20
- J2 pad 36: /GPIO_44 -> /GPIO_24
- J2 pad 39: /GPIO_13 -> /GPIO_25
- J2 pad 40: /GPIO_45 -> /GPIO_29
- J2 pad 41: /GPIO_14 -> /GPIO_26
- J2 pad 42: /GPIO_46 -> /GPIO_30
- J2 pad 43: /GPIO_15 -> /GPIO_27
- J2 pad 44: /GPIO_47 -> /GPIO_31
- J2 pad 45: /GPIO_16 -> /GPIO_28
- J2 pad 46: /GPIO_48 -> /GPIO_32
- J3 pad 10: /GPIO_52 -> /GPIO_40
- J3 pad 13: /GPIO_21 -> /GPIO_41
- J3 pad 14: /GPIO_53 -> /GPIO_45
- J3 pad 15: /GPIO_22 -> /GPIO_42
- J3 pad 16: /GPIO_54 -> /GPIO_46
- J3 pad 17: /GPIO_23 -> /GPIO_43
- J3 pad 18: /GPIO_55 -> /GPIO_47
- J3 pad 19: /GPIO_24 -> /GPIO_44
- J3 pad 20: /GPIO_56 -> /GPIO_48
- J3 pad 23: /GPIO_25 -> /GPIO_49
- J3 pad 24: /GPIO_57 -> /GPIO_53
- J3 pad 25: /GPIO_26 -> /GPIO_50
- J3 pad 26: /GPIO_58 -> /GPIO_54
- J3 pad 27: /GPIO_27 -> /GPIO_51
- J3 pad 28: /GPIO_59 -> /GPIO_55
- J3 pad 29: /GPIO_28 -> /GPIO_52
- J3 pad 3: /GPIO_17 -> /GPIO_33
- J3 pad 30: /GPIO_60 -> /GPIO_56
- J3 pad 33: /GPIO_29 -> /GPIO_57
- J3 pad 35: /GPIO_30 -> /GPIO_58
- J3 pad 37: /GPIO_31 -> /GPIO_59
- J3 pad 39: /GPIO_32 -> /GPIO_60
- J3 pad 4: /GPIO_49 -> /GPIO_37
- J3 pad 5: /GPIO_18 -> /GPIO_34
- J3 pad 6: /GPIO_50 -> /GPIO_38
- J3 pad 7: /GPIO_19 -> /GPIO_35
- J3 pad 8: /GPIO_51 -> /GPIO_39
- J3 pad 9: /GPIO_20 -> /GPIO_36
- J4 pad 3: /QSPI_CS -> /QSPI_SS
- R25 pad 1: /CBSEL0 -> Net-(D7-K)
- R25 pad 2: Net-(JP1-A) -> GND
- U2 pad A1: /GPIO_34 -> /GPIO_6
- U2 pad A10: unconnected-(U2-IOT_170-PadA10) -> /GPIO_38
- U2 pad A11: unconnected-(U2-IOT_168-PadA11) -> /GPIO_39
- U2 pad A2: /GPIO_33 -> /GPIO_5
- U2 pad A5: /GPIO_12 -> /GPIO_20
- U2 pad A6: /GPIO_24 -> /GPIO_44
- U2 pad A7: /GPIO_21 -> /GPIO_41
- U2 pad A8: /GPIO_20 -> /GPIO_36
- U2 pad A9: /GPIO_27 -> /GPIO_51
- U2 pad B11: unconnected-(U2-IOR_161-PadB11) -> /GPIO_40
- U2 pad B3: /GPIO_32 -> /GPIO_60
- U2 pad B5: /GPIO_25 -> /GPIO_49
- U2 pad B6: /GPIO_23 -> /GPIO_43
- U2 pad B7: /GPIO_22 -> /GPIO_42
- U2 pad B8: /GPIO_19 -> /GPIO_35
- U2 pad B9: /GPIO_28 -> /GPIO_52
- U2 pad C11: unconnected-(U2-IOR_160-PadC11) -> /GPIO_45
- U2 pad C3: /GPIO_6 -> /GPIO_10
- U2 pad C5: /GNDPLL -> GND
- U2 pad C7: /GPIO_26 -> /GPIO_50
- U2 pad C8: /GPIO_30 -> /GPIO_58
- U2 pad C9: /GPIO_31 -> /GPIO_59
- U2 pad D1: /GPIO_7 -> /GPIO_11
- U2 pad D10: unconnected-(U2-IOR_154-PadD10) -> /GPIO_47
- U2 pad D11: unconnected-(U2-IOR_152-PadD11) -> /GPIO_48
- U2 pad D2: /GPIO_5 -> /GPIO_9
- U2 pad D3: /GPIO_10 -> /GPIO_18
- U2 pad D5: /GPIO_29 -> /GPIO_57
- U2 pad D7: unconnected-(U2-IOT_181-PadD7) -> /GPIO_37
- U2 pad D9: unconnected-(U2-IOR_147-PadD9) -> /GPIO_46
- U2 pad E1: /GPIO_8 -> /GPIO_12
- U2 pad E11: unconnected-(U2-IOR_148-PadE11) -> /GPIO_55
- U2 pad E2: /GPIO_9 -> /GPIO_17
- U2 pad E3: /GPIO_11 -> /GPIO_19
- U2 pad E8: unconnected-(U2-IOR_146-PadE8) -> /GPIO_53
- U2 pad E9: unconnected-(U2-IOR_144-PadE9) -> /GPIO_54
- U2 pad F1: /GPIO_13 -> /GPIO_25
- U2 pad F10: unconnected-(U2-IOR_136-PadF10) -> /GPIO_61
- U2 pad F2: unconnected-(U2-IOL_12B-PadF2) -> /GPIO_13
- U2 pad F3: /GPIO_14 -> /GPIO_26
- U2 pad F4: unconnected-(U2-IOL_13A-PadF4) -> /GPIO_14
- U2 pad F9: unconnected-(U2-IOR_137-PadF9) -> /GPIO_56
- U2 pad G1: /GPIO_16 -> /GPIO_28
- U2 pad G10: unconnected-(U2-IOR_120-PadG10) -> /GPIO_63
- U2 pad G11: unconnected-(U2-IOR_129-PadG11) -> /GPIO_64
- U2 pad G2: /GPIO_17 -> /GPIO_33
- U2 pad G3: /GPIO_15 -> /GPIO_27
- U2 pad G8: unconnected-(U2-IOR_118-PadG8) -> /GPIO_62
- U2 pad H1: /GPIO_35 -> /GPIO_7
- U2 pad H2: /GPIO_18 -> /GPIO_34
- U2 pad H3: unconnected-(U2-IOL_17B-PadH3) -> /GPIO_15
- U2 pad J1: /GPIO_36 -> /GPIO_8
- U2 pad J2: unconnected-(U2-IOL_25B-PadJ2) -> /GPIO_16
- U2 pad J3: /LED2 -> /LED1
- U2 pad J4: /LED1 -> /LED0
- U2 pad J5: unconnected-(U2-IOB_78-PadJ5) -> /LED2
- U2 pad K1: unconnected-(U2-IOL_23B-PadK1) -> /GPIO_21
- U2 pad K2: unconnected-(U2-IOL_25A-PadK2) -> /GPIO_22
- U2 pad K3: unconnected-(U2-IOB_63-PadK3) -> /GPIO_29
- U2 pad K4: unconnected-(U2-IOB_73-PadK4) -> /GPIO_32
- U2 pad K5: unconnected-(U2-IOB_79-PadK5) -> /LED3
- U2 pad L1: unconnected-(U2-IOB_56-PadL1) -> /GPIO_23
- U2 pad L2: unconnected-(U2-IOB_61-PadL2) -> /GPIO_24
- U2 pad L3: unconnected-(U2-IOB_71-PadL3) -> /GPIO_30
- U2 pad L4: unconnected-(U2-IOB_72-PadL4) -> /GPIO_31
- U2 pad L6: /GNDPLL -> GND
Other:
- board text added: "LED2"
- board text added: "LED3"
- board text removed: "NextMicon"
