File: boards/cherry/board/src/cherry.kicad_sch (KiCad schematic)
At the start: 69 parts, among them J1 TYPE-C-31-M-12, J2 PinHeader_2x24_Duplicate, J3 PinHeader_2x24_Duplicate, J5 SPI PROGRAM, SW1 TS-1187A-B-A-B, SW3 USER, U2 W25Q32JVSSIQ, U3 ICE40HX8K-BG121, U4 TPS62A02APDDCR, U5 TPS62A02APDDCR, X1 OXETDLJANF-48.000000MHz

Commit message: wip
Parts:
- removed JP2: IMAGE1, Jumper:SolderJumper-2_P1.3mm_Open_RoundedPad1.0x1.5mm, symbol Jumper:SolderJumper_2_Open
- removed R25, R26: 1k, Cherry:R_0402_1005Metric, symbol Cherry:R
- J2, J3: value PinHeader_2x24_Duplicate -> PinHeader_2x24; symbol Cherry:PinHeader_1x24 -> Cherry:PinHeader_2x24_Paired; now fitted
- JP1: value IMAGE0 -> USER
- renumbered J5 to J4, SW3 to SW2
Connections:
- net +3V3: now also D1.2 (A), R17.1; no longer R17.2, R19.1
- net +5V: now also D5.5 (VBUS)
- net CBSEL0: now also JP1.1 (A)
- net GND: now also R19.2, R21.2, R22.2, R29.2; no longer D1.1 (K), D3.1 (K), D4.1 (K), D6.1 (K)
- net LED0: no longer R21.1
- net LED1: no longer R22.1
- net PROG_LED: no longer R29.1
- net USB_DM_ESD: now also D5.4 (I/O2); no longer D5.6 (I/O1)
- net USB_DP_ESD: now also D5.6 (I/O1), R16.1; no longer D5.4 (I/O2)
- net USB_DP_FPGA: no longer R16.2
- net USB_PULLUP: no longer R16.1
- net at D3.2 (A): no longer R21.2
- net at D4.2 (A): no longer R22.2
- net at D6.2 (A): no longer R29.2
- net CRESET_B renamed CRESET
- net CRESET: now also R17.2; no longer R17.1
- net QSPI_CS_B renamed QSPI_SS
- net QSPI_SS: no longer J4.3 (Pin_3)
- net USB_DM renamed USB_DM_PIN
- net USB_DM_PIN: now also D5.3 (I/O2); no longer D5.1 (I/O1)
- net USB_DP renamed USB_DP_PIN
- net USB_DP_PIN: now also D5.1 (I/O1); no longer D5.3 (I/O2)
- net VBUS: no longer names the net of FB1.2, J1.A4 (VBUS), J1.A9 (VBUS), J1.B4 (VBUS), J1.B9 (VBUS)
- net VBUS: no longer D5.5 (VBUS)
- new net: D3.1 (K), R21.1
- new net: D1.1 (K), R19.1
- new net: D4.1 (K), R22.1
- new net: D6.1 (K), R29.1
- new net QSPI_CS: J4.3 (Pin_3)
- new net USB_PU_FPGA: R16.2
Other:
- note added: "Decoupling"
- note removed: "Decoupling - iCE40"
- note removed: "IMAGE 1:0 (BRIDGE = 1)"
- note removed: "MODE / PROG"
- note removed: "Native USB - FPGA Full Speed"
- note removed: "RESET (rail power-cycle)"
- moved on the sheet: C1, C10, C11, C16, C17, C18, C19, C2, C20, C21, C22, C23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

Commit message: r
Parts:
- R9: value 100k -> 10k
Changed lines of the file:
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@@
 			)
 		)
-		(property "Value" "100k"
+		(property "Value" "10k"
 			(at 205.105 205.74 0)
 			(show_name no)

Commit message: wip
Parts:
- added JP2: USER, Cherry:SolderJumper-2_P1.3mm_Open_RoundedPad1.0x1.5mm, symbol Jumper:SolderJumper_2_Open
- J2, J3: value PinHeader_2x24 -> Conn_02x24_Odd_Even; footprint Cherry:PinHeader_2x24_P2.54mm_Duplicate -> Connector_PinHeader_2.54mm:PinHeader_2x24_P2.54mm_Vertical; symbol Cherry:PinHeader_2x24_Paired -> Connector_Generic:Conn_02x24_Odd_Even
- J4: footprint Cherry:PinHeader_1x06_P2.54mm -> Connector_PinHeader_2.54mm:PinHeader_1x06_P2.54mm_Vertical; symbol Cherry:PinHeader_1x06 -> Connector_Generic:Conn_01x06; now fitted
- JP1: footprint Jumper:SolderJumper-2_P1.3mm_Open_RoundedPad1.0x1.5mm -> Cherry:SolderJumper-2_P1.3mm_Open_RoundedPad1.0x1.5mm
- renumbered C27 to C1, C16 to C12, C17 to C13, C6 to C14, C18 to C15, C19 to C16, C7 to C17, C20 to C18, C21 to C19, C28 to C2, C22 to C20, C23 to C21, C24 to C22, C25 to C23, C1 to C3, C3 to C4, C2 to C5, C4 to C6, C29 to C7, D5 to D1, D1 to D2, D6 to D5, R13 to R1, R5 to R10, R6 to R11, R1 to R12, R2 to R13, R3 to R14, R9 to R15, R27 to R16, R4 to R17, R19 to R18, R21 to R19, R10 to R2, R22 to R20, R29 to R21, R23 to R22, R24 to R23, R8 to R3, R11 to R4, R17 to R5, R12 to R6, R14 to R7, R15 to R8, R16 to R9, U2 to U1, U3 to U2, U4 to U3, U5 to U4
Connections:
- net PROG_LED is gone; now on net PROG: U2.J10 (IOR_117)
- net USB_PU_FPGA is gone; now on net USB_PU: R9.2
- net +3V3: now also J2.18 (Pin_18), J2.28 (Pin_28), J2.3 (Pin_3), J2.38 (Pin_38), J2.4 (Pin_4), J2.48 (Pin_48), J2.8 (Pin_8), J3.12 (Pin_12), J3.2 (Pin_2), J3.22 (Pin_22), J3.32 (Pin_32), J3.42 (Pin_42), J3.45 (Pin_45), J3.46 (Pin_46), JP2.2 (B); no longer J2.2, J3.23
- net +5V: now also J2.2 (Pin_2), J3.47 (Pin_47), J3.48 (Pin_48); no longer J3.24
- net CBSEL1: now also JP2.1 (A)
- net CRESET: now also J2.5 (Pin_5); no longer J2.6
- net GND: now also J2.17 (Pin_17), J2.27 (Pin_27), J2.37 (Pin_37), J2.47 (Pin_47), J2.7 (Pin_7), J3.1 (Pin_1), J3.11 (Pin_11), J3.31 (Pin_31), J3.41 (Pin_41); no longer J2.3, J2.4, J2.5, J3.19, J3.20, J3.22
- net GPIO_1: now also J2.9 (Pin_9); no longer J2.7
- net GPIO_10: now also J2.31 (Pin_31); no longer J2.16
- net GPIO_11: now also J2.33 (Pin_33); no longer J2.17
- net GPIO_12: now also J2.35 (Pin_35); no longer J2.18
- net GPIO_13: now also J2.39 (Pin_39); no longer J2.19
- net GPIO_14: now also J2.41 (Pin_41); no longer J2.20
- net GPIO_15: now also J2.43 (Pin_43); no longer J2.21
- net GPIO_16: now also J2.45 (Pin_45); no longer J2.22
- net GPIO_17: now also J3.3 (Pin_3); no longer J2.23
- net GPIO_18: now also J3.5 (Pin_5); no longer J2.24
- net GPIO_19: now also J3.7 (Pin_7); no longer J3.1
- net GPIO_2: now also J2.11 (Pin_11); no longer J2.8
- net GPIO_20: now also J3.9 (Pin_9); no longer J3.2
- net GPIO_21: now also J3.13 (Pin_13); no longer J3.3
- net GPIO_22: now also J3.15 (Pin_15); no longer J3.4
- net GPIO_23: now also J3.17 (Pin_17); no longer J3.5
- net GPIO_24: now also J3.19 (Pin_19); no longer J3.6
- net GPIO_25: now also J3.23 (Pin_23); no longer J3.7
- net GPIO_26: now also J3.25 (Pin_25); no longer J3.8
- net GPIO_27: now also J3.27 (Pin_27); no longer J3.9
- net GPIO_28: now also J3.29 (Pin_29); no longer J3.10
- net GPIO_29: now also J3.33 (Pin_33); no longer J3.11
- net GPIO_3: now also J2.13 (Pin_13); no longer J2.9
- net GPIO_30: now also J3.35 (Pin_35); no longer J3.12
- net GPIO_31: now also J3.37 (Pin_37); no longer J3.13
- net GPIO_32: now also J3.39 (Pin_39); no longer J3.14
- net GPIO_33: now also J2.10 (Pin_10); no longer J3.15
- net GPIO_34: now also J2.12 (Pin_12); no longer J3.16
- net GPIO_35: now also J2.14 (Pin_14); no longer J3.17
- net GPIO_36: now also J2.16 (Pin_16); no longer J3.18
- net GPIO_4: now also J2.15 (Pin_15); no longer J2.10
- net GPIO_5: now also J2.19 (Pin_19); no longer J2.11
- net GPIO_6: now also J2.21 (Pin_21); no longer J2.12
- net GPIO_7: now also J2.23 (Pin_23); no longer J2.13
- net GPIO_8: now also J2.25 (Pin_25); no longer J2.14
- net GPIO_9: now also J2.29 (Pin_29); no longer J2.15
- net LED0: now also D4.2 (A)
- net LED1: now also D5.2 (A)
- net CC1: now reaches J1.A5 (CC1), R10.1
- net FB3V3: now reaches R12.2, R13.1, U3.6 (FB)
- net GPIO_52: now reaches J3.10 (Pin_10)
- net GPIO_53: now reaches J3.14 (Pin_14)
- net GPIO_54: now reaches J3.16 (Pin_16)
- net GPIO_55: now reaches J3.18 (Pin_18)
- net GPIO_56: now reaches J3.20 (Pin_20)
- net GPIO_57: now reaches J3.24 (Pin_24)
- net GPIO_49: now reaches J3.4 (Pin_4)
- net GPIO_50: now reaches J3.6 (Pin_6)
- net GPIO_51: now reaches J3.8 (Pin_8)
- net VBUD: now reaches FB1.2, J1.A4 (VBUS), J1.A9 (VBUS), J1.B4 (VBUS), J1.B9 (VBUS)
- net PROG: now reaches D3.2 (A)
- net GPIO_37: now reaches J2.20 (Pin_20)
- net GPIO_38: now reaches J2.22 (Pin_22)
- net GPIO_39: now reaches J2.24 (Pin_24)
- net CC2: now reaches J1.B5 (CC2), R11.1
- net FB1V2: now reaches R14.2, R17.1, U4.6 (FB)
- net PWR_EN renamed PWRSW
- net USB_DM_ESD renamed USB_ESD_DM
- net USB_DM_FPGA renamed USB_DM
- net USB_DM_PIN renamed USB_PIN_DM
- net USB_DP_ESD renamed USB_ESD_DP
- net USB_DP_FPGA renamed USB_DP
- net USB_DP_PIN renamed USB_PIN_DP
- net USB_PULLUP renamed USB_PU
- net USER_BTN renamed BTN
- new net GPIO_40: J2.26 (Pin_26)
- new net GPIO_41: J2.30 (Pin_30)
- new net GPIO_42: J2.32 (Pin_32)
- new net GPIO_43: J2.34 (Pin_34)
- new net GPIO_44: J2.36 (Pin_36)
- new net GPIO_45: J2.40 (Pin_40)
- new net GPIO_46: J2.42 (Pin_42)
- new net GPIO_47: J2.44 (Pin_44)
- new net GPIO_48: J2.46 (Pin_46)
- new net GPIO_58: J3.26 (Pin_26)
- new net GPIO_59: J3.28 (Pin_28)
- new net GPIO_60: J3.30 (Pin_30)
- new net GPIO_61: J3.34 (Pin_34)
- new net GPIO_62: J3.36 (Pin_36)
- new net GPIO_63: J3.38 (Pin_38)
- new net GPIO_64: J3.40 (Pin_40)
- now unconnected: U2.D11 (IOR_152), U2.E11 (IOR_148), U2.E9 (IOR_144), U2.F10 (IOR_136), U2.F11 (IOR_140_GBIN3), U2.F2 (IOL_12B), U2.F4 (IOL_13A), U2.F9 (IOR_137), U2.G10 (IOR_120), U2.G11 (IOR_129), U2.H10 (IOR_116), U2.H11 (IOR_119), U2.H3 (IOL_17B), U2.H7 (IOB_87), U2.J11 (IOR_114), U2.J5 (IOB_78), U2.J7 (IOB_86), U2.K1 (IOL_23B), U2.K11 (IOR_115), U2.K2 (IOL_25A), U2.K3 (IOB_63), U2.K4 (IOB_73), U2.K5 (IOB_79), U2.K7 (IOB_89), U2.L1 (IOB_56), U2.L2 (IOB_61), U2.L3 (IOB_71), U2.L4 (IOB_72), U2.L5 (IOB_81_GBIN5), U2.L7 (IOB_94)
- no-connect marks 16 -> 46
Other:
- note added: "BootSelect"
- moved on the sheet: C7, D2, D3, D4, D5, JP1, R15, R16, R18, R19, R20, R21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

Commit message: chore
Parts:
- added C24: 100nF, Cherry:C_0402_1005Metric, symbol Cherry:C
- added D6, D7: KT-0603R, Cherry:LED_0603_1608Metric, symbol Cherry:LED
- added R24, R25: 1k, Cherry:R_0402_1005Metric, symbol Cherry:R
- R14: renamed from R6; value 1k -> 10k
- renumbered R10 to R1, R2 to R10, R3 to R11, R4 to R12, R5 to R13, R1 to R15, R22 to R16, R23 to R17, R11 to R2, R15 to R22, R16 to R23, R12 to R3, R13 to R4, R14 to R5, R17 to R6, R9 to R7, R7 to R8, R8 to R9
Connections:
- net GNDPLL is gone; now on net GND: C1.2, C2.2, U2.C5 (GNDPLL1), U2.L6 (GNDPLL0)
- net QSPI_CS is gone; now on net QSPI_SS: J4.3 (Pin_3)
- net BTN: now also C24.1
- net GND: now also C24.2, R24.2, R25.2
- net GPIO_10: now also J2.21 (Pin_21), U2.C3 (IOL_4B); no longer J2.31 (Pin_31), U2.D3 (IOL_9B)
- net GPIO_11: now also J2.23 (Pin_23), U2.D1 (IOL_8B); no longer J2.33 (Pin_33), U2.E3 (IOL_10B)
- net GPIO_12: now also J2.25 (Pin_25), U2.E1 (IOL_8A); no longer J2.35 (Pin_35), U2.A5 (IOT_207)
- net GPIO_13: now also J2.20 (Pin_20), U2.F2 (IOL_12B); no longer J2.39 (Pin_39), U2.F1 (IOL_12A)
- net GPIO_14: now also J2.22 (Pin_22), U2.F4 (IOL_13A); no longer J2.41 (Pin_41), U2.F3 (IOL_13B_GBIN7)
- net GPIO_15: now also J2.24 (Pin_24), U2.H3 (IOL_17B); no longer J2.43 (Pin_43), U2.G3 (IOL_17A)
- net GPIO_16: now also J2.26 (Pin_26), U2.J2 (IOL_25B); no longer J2.45 (Pin_45), U2.G1 (IOL_14A_GBIN6)
- net GPIO_17: now also J2.29 (Pin_29), U2.E2 (IOL_10A); no longer J3.3 (Pin_3), U2.G2 (IOL_14B)
- net GPIO_18: now also J2.31 (Pin_31), U2.D3 (IOL_9B); no longer J3.5 (Pin_5), U2.H2 (IOL_18B)
- net GPIO_19: now also J2.33 (Pin_33), U2.E3 (IOL_10B); no longer J3.7 (Pin_7), U2.B8 (IOT_177)
- net GPIO_20: now also J2.35 (Pin_35), U2.A5 (IOT_207); no longer J3.9 (Pin_9), U2.A8 (IOT_190)
- net GPIO_21: now also J2.30 (Pin_30), U2.K1 (IOL_23B); no longer J3.13 (Pin_13), U2.A7 (IOT_192)
- net GPIO_22: now also J2.32 (Pin_32), U2.K2 (IOL_25A); no longer J3.15 (Pin_15), U2.B7 (IOT_197_GBIN1)
- net GPIO_23: now also J2.34 (Pin_34), U2.L1 (IOB_56); no longer J3.17 (Pin_17), U2.B6 (IOT_198_GBIN0)
- net GPIO_24: now also J2.36 (Pin_36), U2.L2 (IOB_61); no longer J3.19 (Pin_19), U2.A6 (IOT_206)
- net GPIO_25: now also J2.39 (Pin_39), U2.F1 (IOL_12A); no longer J3.23 (Pin_23), U2.B5 (IOT_208)
- net GPIO_26: now also J2.41 (Pin_41), U2.F3 (IOL_13B_GBIN7); no longer J3.25 (Pin_25), U2.C7 (IOT_191)
- net GPIO_27: now also J2.43 (Pin_43), U2.G3 (IOL_17A); no longer J3.27 (Pin_27), U2.A9 (IOT_178)
- net GPIO_28: now also J2.45 (Pin_45), U2.G1 (IOL_14A_GBIN6); no longer J3.29 (Pin_29), U2.B9 (IOT_174)
- net GPIO_29: now also J2.40 (Pin_40), U2.K3 (IOB_63); no longer J3.33 (Pin_33), U2.D5 (IOT_212)
- net GPIO_30: now also J2.42 (Pin_42), U2.L3 (IOB_71); no longer J3.35 (Pin_35), U2.C8 (IOT_179)
- net GPIO_31: now also J2.44 (Pin_44), U2.L4 (IOB_72); no longer J3.37 (Pin_37), U2.C9 (IOT_172)
- net GPIO_32: now also J2.46 (Pin_46), U2.K4 (IOB_73); no longer J3.39 (Pin_39), U2.B3 (IOT_221)
- net GPIO_33: now also J3.3 (Pin_3), U2.G2 (IOL_14B); no longer J2.10 (Pin_10), U2.A2 (IOT_222)
- net GPIO_34: now also J3.5 (Pin_5), U2.H2 (IOL_18B); no longer J2.12 (Pin_12), U2.A1 (IOT_225)
- net GPIO_35: now also J3.7 (Pin_7), U2.B8 (IOT_177); no longer J2.14 (Pin_14), U2.H1 (IOL_18A)
- net GPIO_36: now also J3.9 (Pin_9), U2.A8 (IOT_190); no longer J2.16 (Pin_16), U2.J1 (IOL_23A)
- net GPIO_37: now also J3.4 (Pin_4), U2.D7 (IOT_181); no longer J2.20 (Pin_20)
- net GPIO_38: now also J3.6 (Pin_6), U2.A10 (IOT_170); no longer J2.22 (Pin_22)
- net GPIO_39: now also J3.8 (Pin_8), U2.A11 (IOT_168); no longer J2.24 (Pin_24)
- net GPIO_40: now also J3.10 (Pin_10), U2.B11 (IOR_161); no longer J2.26 (Pin_26)
- net GPIO_41: now also J3.13 (Pin_13), U2.A7 (IOT_192); no longer J2.30 (Pin_30)
- net GPIO_42: now also J3.15 (Pin_15), U2.B7 (IOT_197_GBIN1); no longer J2.32 (Pin_32)
- net GPIO_43: now also J3.17 (Pin_17), U2.B6 (IOT_198_GBIN0); no longer J2.34 (Pin_34)
- net GPIO_44: now also J3.19 (Pin_19), U2.A6 (IOT_206); no longer J2.36 (Pin_36)
- net GPIO_45: now also J3.14 (Pin_14), U2.C11 (IOR_160); no longer J2.40 (Pin_40)
- net GPIO_46: now also J3.16 (Pin_16), U2.D9 (IOR_147); no longer J2.42 (Pin_42)
- net GPIO_47: now also J3.18 (Pin_18), U2.D10 (IOR_154); no longer J2.44 (Pin_44)
- net GPIO_48: now also J3.20 (Pin_20), U2.D11 (IOR_152); no longer J2.46 (Pin_46)
- net GPIO_49: now also J3.23 (Pin_23), U2.B5 (IOT_208); no longer J3.4 (Pin_4)
- net GPIO_5: now also J2.10 (Pin_10), U2.A2 (IOT_222); no longer J2.19 (Pin_19), U2.D2 (IOL_9A)
- net GPIO_50: now also J3.25 (Pin_25), U2.C7 (IOT_191); no longer J3.6 (Pin_6)
- net GPIO_51: now also J3.27 (Pin_27), U2.A9 (IOT_178); no longer J3.8 (Pin_8)
- net GPIO_52: now also J3.29 (Pin_29), U2.B9 (IOT_174); no longer J3.10 (Pin_10)
- net GPIO_53: now also J3.24 (Pin_24), U2.E8 (IOR_146); no longer J3.14 (Pin_14)
- net GPIO_54: now also J3.26 (Pin_26), U2.E9 (IOR_144); no longer J3.16 (Pin_16)
- net GPIO_55: now also J3.28 (Pin_28), U2.E11 (IOR_148); no longer J3.18 (Pin_18)
- net GPIO_56: now also J3.30 (Pin_30), U2.F9 (IOR_137); no longer J3.20 (Pin_20)
- net GPIO_57: now also J3.33 (Pin_33), U2.D5 (IOT_212); no longer J3.24 (Pin_24)
- net GPIO_58: now also J3.35 (Pin_35), U2.C8 (IOT_179); no longer J3.26 (Pin_26)
- net GPIO_59: now also J3.37 (Pin_37), U2.C9 (IOT_172); no longer J3.28 (Pin_28)
- net GPIO_6: now also J2.12 (Pin_12), U2.A1 (IOT_225); no longer J2.21 (Pin_21), U2.C3 (IOL_4B)
- net GPIO_60: now also J3.39 (Pin_39), U2.B3 (IOT_221); no longer J3.30 (Pin_30)
- net GPIO_61: now also U2.F10 (IOR_136)
- net GPIO_62: now also U2.G8 (IOR_118)
- net GPIO_63: now also U2.G10 (IOR_120)
- net GPIO_64: now also U2.G11 (IOR_129)
- net GPIO_7: now also J2.14 (Pin_14), U2.H1 (IOL_18A); no longer J2.23 (Pin_23), U2.D1 (IOL_8B)
- net GPIO_8: now also J2.16 (Pin_16), U2.J1 (IOL_23A); no longer J2.25 (Pin_25), U2.E1 (IOL_8A)
- net GPIO_9: now also J2.19 (Pin_19), U2.D2 (IOL_9A); no longer J2.29 (Pin_29), U2.E2 (IOL_10A)
- net LED2: now reaches U2.J5 (IOB_78)
- net LED2: now also D6.2 (A)
- net LED3: now reaches U2.K5 (IOB_79)
- net LED3: now also D7.2 (A)
- net VBUD renamed VBUS
- new net: D7.1 (K), R25.1
- new net: D6.1 (K), R24.1
- no-connect marks 46 -> 19
Other:
- moved on the sheet: D2, D3, D4, D5, R10, R11, R12, R13, R14, R18, R19, R20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

Commit message: wip
Parts:
- U1: symbol Cherry:W25Q32JVSSIM -> Cherry:W25Q32JVSSIQ
Connections:
- net BTN: now also U2.F11 (IOR_140_GBIN3); no longer U2.C4 (IOL_4A)
- net CRESET: now also SW1.1
- net GND: no longer C1.2, C2.2, U2.C5 (GNDPLL1), U2.L6 (GNDPLL0)
- net GPIO_43: now also U2.H10 (IOR_116); no longer U2.B6 (IOT_198_GBIN0)
- net PWRSW: no longer SW1.1
- net PLL0_IN: now reaches J3.43 (Pin_43)
- net PLL0_IN: now also U2.L5 (IOB_81_GBIN5)
- net PLL1_IN: now reaches J3.44 (Pin_44)
- net PLL1_IN: now also U2.B6 (IOT_198_GBIN0)
- new net GNDPLL: C1.2, C2.2, U2.C5 (GNDPLL1), U2.L6 (GNDPLL0)
- no-connect marks 19 -> 15
Changed lines of the file:
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@@
 	)
 	(junction
-		(at 152.4 212.09)
-		(diameter 0)
-		(color 0 0 0 0)
-	)
-	(junction
 		(at 31.75 50.8)
 		(diameter 0)
@@
 		(at 59.69 144.78)
 	)
-	(no_connect
-		(at 387.35 156.21)
+	(label "PLL1_IN"
+		(at 387.35 156.21 180)
+		(effects
+			(font
+				(size 1.27 1.27)
+			)
+			(justify right bottom)
+		)
 	)
 	(no_connect
@@
 		(at 312.42 101.6)
 	)
-	(no_connect
-		(at 312.42 104.14)
+	(label "GPIO_43"
+		(at 312.42 104.14 0)
+		(effects
+			(font
+				(size 1.27 1.27)
+			)
+			(justify left bottom)
+		)
 	)
 	(no_connect
 		(at 312.42 106.68)
 	)
-	(no_connect
-		(at 312.42 119.38)
-	)
-	(no_connect
-		(at 312.42 152.4)
+	(label "PLL0_IN"
+		(at 312.42 152.4 0)
+		(effects
+			(font
+				(size 1.27 1.27)
+			)
+			(justify left bottom)
+		)
 	)
 	(no_connect
@@
 		(at 312.42 162.56)
 	)
-	(no_connect
-		(at 374.65 156.21)
+	(label "PLL0_IN"
+		(at 374.65 156.21 180)
+		(effects
+			(font
+				(size 1.27 1.27)
+			)
+			(justify right bottom)
+		)
 	)
 	(wire
@@
 		)
 	)
+	(no_connect
+		(at 271.78 124.46)
+	)
 	(wire
 		(pts
-			(xy 256.54 124.46) (xy 271.78 124.46)
+			(xy 312.42 119.38) (xy 317.5 119.38)
 		)
 		(stroke
@@
 	(wire
 		(pts
-			(xy 152.4 212.09) (xy 152.4 214.63)
+			(xy 144.78 214.63) (xy 152.4 214.63)
 		)
 		(stroke
@@
 	(wire
 		(pts
-			(xy 228.6 55.88) (xy 228.6 58.42)
-		)
-		(stroke
-			(width 0)
-			(type default)
-		)
-	)
-	(wire
-		(pts
 			(xy 171.45 76.2) (xy 271.78 76.2)
 		)
@@
 	)
 	(label "BTN"
-		(at 256.54 124.46 0)
+		(at 317.5 119.38 0)
 		(effects
 			(font
@@
 		)
 	)
+	(label "CRESET"
+		(at 144.78 214.63 0)
+		(effects
+			(font
+				(size 1.27 1.27)
+			)
+			(justify left bottom)
+		)
+	)
 	(label "LED0"
 		(at 256.54 119.38 0)
@@
 		)
 	)
+	(label "GNDPLL"
+		(at 264.16 55.88 180)
+		(effects
+			(font
+				(size 1.27 1.27)
+			)
+			(justify right bottom)
+		)
+	)
 	(label "QSPI_SCK"
 		(at 171.45 71.12 0)
@@
 		)
 	)
-	(label "GPIO_43"
+	(label "PLL1_IN"
 		(at 317.5 45.72 0)
 		(effects
@@
 	)
 	(symbol
-		(lib_id "Cherry:GND")
-		(at 228.6 58.42 0)
+		(lib_id "Cherry:PWR_FLAG")
+		(at 228.6 55.88 0)
 		(unit 1)
 		(body_style 1)
@@
 		(in_pos_files yes)
 		(dnp no)
-		(property "Reference" "#PWR0709"
-			(at 236.22 44.45 0)
+		(property "Reference" "#FLG0505"
+			(at 228.6 53.975 0)
 			(hide yes)
 			(show_name no)
@@
 			)
 		)
-		(property "Value" "GND"
-			(at 228.6 62.51 0)
+		(property "Value" "PWR_FLAG"
+			(at 228.6 51.435 0)
+			(hide yes)
 			(show_name no)
 			(do_not_autoplace no)
@@
 		)
 		(property "Footprint" ""
-			(at 236.22 46.99 0)
+			(at 228.6 55.88 0)
 			(show_name no)
 			(do_not_autoplace no)
@@
 		)
 		(property "Datasheet" ""
-			(at 236.22 46.99 0)
+			(at 228.6 55.88 0)
 			(show_name no)
 			(do_not_autoplace no)
@@
 		)
 		(property "Description" ""
-			(at 236.22 46.99 0)
+			(at 228.6 55.88 0)
 			(show_name no)
 			(do_not_autoplace no)
@@
 			(project "cherry"
 				(path "/00000000-0000-0000-0000-000000000001"
-					(reference "#PWR0709")
+					(reference "#FLG0505")
 					(unit 1)
 				)
@@
 	)
 	(symbol
-		(lib_id "Cherry:W25Q32JVSSIM")
+		(lib_id "Cherry:W25Q32JVSSIQ")
 		(at 158.75 74.93 0)
 		(unit 1)
